Commit message: added realsense to xacro file

File: boris_description/urdf/boris.urdf.xacro (robot description, xacro)
@@ -5,5 +5,5 @@
   <xacro:include filename="$(find sensors_description)/urdf/rgb_cam.xacro" />
   <xacro:include filename="$(find shark_description)/urdf/shark.xacro" />
-  <xacro:include filename="$(find sensors_description)/urdf/realsense_camera.urdf.xacro" />
+  <xacro:include filename="$(find sensors_description)/urdf/realsense_camera.xacro" />
   <xacro:include filename="$(find boris_head_description)/urdf/boris_head.urdf" />
   <!-- <xacro:include filename="$(find interbotix_xsarm_descriptions)/urdf/wx200.urdf.xacro" /> -->
@@ -103,7 +103,5 @@
     <origin xyz="0 0 ${dorso_height + 0.04}" rpy="0 0 0" />
   </joint>
-  <xacro:realsense_camera name="camera" parent="dorso_link">
-    <origin xyz="${dorso_len/2 + 0.05} 0 ${dorso_height + 0.053}" rpy="0 0 0" />
-  </xacro:realsense_camera>
+  <xacro:realsense_camera name="camera" parent="dorso_link" xyz="${dorso_len/2 + 0.05} 0 ${dorso_height + 0.053}" rpy="0 0 0"/>
   <xacro:dorso parent="base_link" depth="${dorso_len}" width="${dorso_width}" height="${dorso_height}" xyz="${-base_len/2 + (dorso_len/2)} 0 ${base_height/2}" rpy="0 0 0"/>
   <xacro:arm_support parent="dorso_link" width="${arm_support_width}" height="${arm_support_height}" depth="${arm_support_len}" xyz="${dorso_len/2 + arm_support_len/2} 0 ${arm_z_position}" rpy="0 0 0"/>

File: sensors_description/urdf/realsense_camera.xacro (robot description, xacro)
@@ -1,6 +1,6 @@
 <?xml version="1.0"?>
-<robot xmlns:xacro="http://www.ros.org/wiki/xacro">
+<robot name="realsense_rgbd" xmlns:xacro="http://www.ros.org/wiki/xacro">
   <xacro:property name="M_PI" value="3.1415926535897931"/>
-  <xacro:macro name="realsense_camera" params="name parent *origin">
+  <xacro:macro name="realsense_camera" params="name parent xyz rpy">
       <!-- @TODO: GABIARRA PRA GIRAR A CAMERA -->
       <link name="head_pan_link_static">
@@ -34,5 +34,5 @@
       </link>
       <joint name="head_pan_joint_static" type="fixed">
-          <xacro:insert_block name="origin"/>
+          <origin xyz="${xyz}" rpy="${rpy}"/>
           <parent link="${parent}"/>
           <child link="head_pan_link_static"/>
@@ -41,5 +41,5 @@
       </joint>
       <joint name="head_pan_joint" type="revolute">
-          <xacro:insert_block name="origin"/>
+          <origin xyz="${xyz}" rpy="${rpy}"/>
           <parent link="${parent}"/>
           <child link="head_pan_link"/>

File: shark_description/urdf/shark_description.xacro (robot description, xacro)
@@ -58,14 +58,5 @@
   </xacro:macro>
   <xacro:macro name="shark_base">
-    <link name="base_footprint">
-      <xacro:box_inertia m="8" w="0.001" h="0.001" d="0.001" />
-      <visual>
-        <origin xyz="0 0 0" rpy="0 0 0" />
-        <material name="white" />
-        <geometry>
-          <box size="0.001 0.001 0.001" />
-        </geometry>
-      </visual>
-    </link>
+    <link name="base_footprint"/>
     <link name="base_link">
       <xacro:box_inertia m="1" w="${base_len}" h="${base_width}" d="0.01" />

Commit message: changed how arm is included

File: boris_description/urdf/boris.urdf.xacro (robot description, xacro)
@@ -103,4 +103,9 @@
     <origin xyz="0 0 ${dorso_height + 0.04}" rpy="0 0 0" />
   </joint>
+  <joint name="arm_to_robot" type="fixed">
+    <origin xyz="0.1 0 ${arm_support_height/2}" rpy="0 0 0"/>
+    <parent link="arm_support_link"/>
+    <child link="wx200/base_link"/>
+  </joint>
   <xacro:realsense_camera name="camera" parent="dorso_link" xyz="${dorso_len/2 + 0.05} 0 ${dorso_height + 0.053}" rpy="0 0 0"/>
   <xacro:dorso parent="base_link" depth="${dorso_len}" width="${dorso_width}" height="${dorso_height}" xyz="${-base_len/2 + (dorso_len/2)} 0 ${base_height/2}" rpy="0 0 0"/>
@@ -109,5 +114,5 @@
   <xacro:sensor_hokuyo parent="base_link" xyz="${-base_len/2 - 0.017 - 0.024} 0 ${0.02 - base_height/2}" rpy="3.14 0 3.14" name="back"/>
   <xacro:imu parent="base_link" xyz="-0.01 0 ${0.02 - base_height/2}" rpy="-0.014161 -0.0203861 0" />
-  <xacro:boris_arm parent="arm_support_link" xyz="0.1 0 ${arm_support_height/2}" rpy="0 0 0"/>
+  <!-- <xacro:boris_arm parent="arm_support_link" xyz="0.1 0 ${arm_support_height/2}" rpy="0 0 0"/> -->
   <!-- <xacro:rgb_cam parent="wx200/gripper_bar_link" name="webcam" xyz="-0.078 0.0 0.05" rpy="0 0 0"/> -->
   <xacro:shark_base/>
