Commit message: separeted body from base

File: boris_description/urdf/boris.xacro (robot description, xacro)
@@ -3,7 +3,8 @@
   <xacro:include filename="$(find sensors_description)/urdf/hokuyo.xacro" />
   <xacro:include filename="$(find sensors_description)/urdf/sick_lms1xx.xacro" />
-  <!-- <xacro:include filename="$(find sensors_description)/urdf/realsense_camera.urdf.xacro" /> -->
-  <!-- <xacro:include filename="$(find hector_sensors_description)/urdf/realsense_d435_camera.urdf.xacro" /> -->
-  <!-- <xacro:include filename="$(find doris_head_description)/urdf/doris_head.urdf" /> -->
+  <xacro:include filename="$(find sensors_description)/urdf/rgb_cam.xacro" />
+  <xacro:include filename="$(find shark_description)/urdf/shark.xacro" />
+  <xacro:include filename="$(find sensors_description)/urdf/realsense_camera.urdf.xacro" />
+  <xacro:include filename="$(find boris_head_description)/urdf/boris_head.urdf" />
   <!-- <xacro:include filename="$(find interbotix_xsarm_descriptions)/urdf/wx200.urdf.xacro" /> -->
   <xacro:property name="base_width" value="0.336" />
@@ -24,27 +25,4 @@
   <xacro:arg name="arm_z_position" default="0.34"/>
   <xacro:property name="arm_z_position" value="$(arg arm_z_position)" />
-  <!-- <xacro:property name="caster_wheel_radius" value="0.0375"/>
-  <xacro:property name="caster_wheel_joint_offset" value="0.12"/> -->
-  <!-- <xacro:include filename="$(find shark-mb-ros)/urdf/shark_v1_gazebo_plugins.xacro" /> -->
-  <material name="blue">
-    <color rgba="0 0 0.8 1" />
-  </material>
-  <material name="black">
-    <color rgba="0 0 0 1" />
-  </material>
-  <material name="darkgray">
-    <color rgba="0.2 0.2 0.2 1" />
-  </material>
-  <material name="lightgray">
-    <color rgba="0.8 0.8 0.8 1" />
-  </material>
-  <material name="white">
-    <color rgba="1 1 1 1" />
-  </material>
-  <material name="red">
-    <color rgba="0.8 0.0 0.0 1.0" />
-  </material>
-  <!-- Import Rviz colors -->
-  <!--  <xacro:include filename="$(find ros_robotics)/urdf/materials.xacro" /> -->
   <xacro:macro name="box_inertia" params="m w h d">
     <inertial>
@@ -54,68 +32,4 @@
     </inertial>
   </xacro:macro>
-  <link name="base_footprint">
-    <!-- <xacro:box_inertia m="8" w="0.001" h="0.001" d="0.001" /> -->
-    <visual>
-      <origin xyz="0 0 0" rpy="0 0 0" />
-      <material name="white" />
-      <geometry>
-        <box size="0.001 0.001 0.001" />
-      </geometry>
-    </visual>
-  </link>
-  <link name="base_link">
-    <xacro:box_inertia m="1" w="${base_len}" h="${base_width}" d="0.01" />
-    <visual>
-      <material name="lightgray" />
-      <geometry>
-        <box size="${base_len} ${base_width} ${base_height}" />
-      </geometry>
-    </visual>
-    <collision>
-      <geometry>
-        <box size="${base_len} ${base_width} ${base_height}" />
-      </geometry>
-    </collision>
-  </link>
-  <joint name="base_link_joint" type="fixed">
-    <origin xyz="0 0 ${base_height/2 + caster_height}" rpy="0 0 0" />
-    <parent link="base_footprint" />
-    <child link="base_link" />
-  </joint>
-  <xacro:macro name="cylinder_inertia" params="m r h">
-    <inertial>
-      <mass value="${m}" />
-      <inertia ixx="${m*(3*r*r+h*h)/12}" ixy="0" ixz="0" iyy="${m*(3*r*r+h*h)/12}" iyz="0"
-        izz="${m*r*r/2}" />
-    </inertial>
-  </xacro:macro>
-  <xacro:macro name="wheel" params="prefix reflect">
-    <link name="${prefix}_wheel">
-      <visual>
-        <material name="darkgray" />
-        <origin xyz="0 0 0" rpy="${pi/2} 0 0" />
-        <geometry>
-          <cylinder radius="${wheel_radius}" length="${wheel_width}" />
-        </geometry>
-      </visual>
-      <collision>
-        <origin xyz="0 0 0" rpy="${pi/2} 0 0" />
-        <geometry>
-          <cylinder radius="${wheel_radius}" length="0.05" />
-        </geometry>
-      </collision>
-      <xacro:cylinder_inertia m="10" r="${wheel_radius}" h="0.05" />
-    </link>
-    <joint name="${prefix}_wheel" type="continuous">
-      <axis xyz="0 1 0" rpy="0 0 0" />
-      <parent link="base_link" />
-      <child link="${prefix}_wheel" />
-      <origin
-        xyz="${wheel_joint_offset} ${((base_width/2)+base_wheel_gap)*reflect} ${(wheel_radius - caster_height) - base_height/2}"
-        rpy="0 0 0" />
-    </joint>
-  </xacro:macro>
-  <xacro:wheel prefix="left" reflect="1" />
-  <xacro:wheel prefix="right" reflect="-1" />
   <xacro:macro name="sphere_inertia" params="m r">
     <inertial>
@@ -179,43 +93,4 @@
     </joint>
   </xacro:macro>
-  <xacro:macro name="rgb_cam" params="parent name xyz rpy">
-    <link name="${name}_link">
-      <visual>
-        <material name="lightgray"/>
-        <geometry>
-          <box size="0.013 0.0627 0.02597"/>
-        </geometry>
-      </visual>
-      <collision>
-        <geometry>
-          <box size="0.013 0.0627 0.02597"/>
-        </geometry>
-      </collision>
-    </link>
-    <link name="${name}_lens_link">
-      <visual>
-        <material name="black"/>
-        <origin xyz="0.001 0 0" rpy="0.0 1.5707963267948966 0.0"/>
-        <geometry>
-          <cylinder radius="0.00725" length="0.013"/>
-        </geometry>
-      </visual>
-      <collision>
-        <geometry>
-          <cylinder radius="0.00725" length="0.013"/>
-        </geometry>
-      </collision>
-    </link>
-    <joint name="${name}_joint" type="fixed">
-      <parent link="${parent}"/>
-      <child link="${name}_link"/>
-      <origin xyz="${xyz}" rpy="${rpy}"/>
-    </joint>
-    <joint name="${name}_lens_joint" type="fixed">
-      <parent link="${name}_link"/>
-      <child link="${name}_lens_link"/>
-      <origin xyz="0.0 -0.015375 0.0"/>
-    </joint>
-  </xacro:macro>
   <joint name="laser_joint" type="fixed">
     <origin xyz="${base_len/2 + 0.017 + 0.05} 0 ${0.02 + base_height/2}" rpy="0 0 0" />
@@ -228,7 +103,7 @@
     <origin xyz="0 0 ${dorso_height + 0.04}" rpy="0 0 0" />
   </joint>
-  <!-- <xacro:realsense_camera name="camera" parent="dorso_link">
+  <xacro:realsense_camera name="camera" parent="dorso_link">
     <origin xyz="${dorso_len/2 + 0.05} 0 ${dorso_height + 0.053}" rpy="0 0 0" />
-  </xacro:realsense_camera> -->
+  </xacro:realsense_camera>
   <xacro:dorso parent="base_link" depth="${dorso_len}" width="${dorso_width}" height="${dorso_height}" xyz="${-base_len/2 + (dorso_len/2)} 0 ${base_height/2}" rpy="0 0 0"/>
   <xacro:arm_support parent="dorso_link" width="${arm_support_width}" height="${arm_support_height}" depth="${arm_support_len}" xyz="${dorso_len/2 + arm_support_len/2} 0 ${arm_z_position}" rpy="0 0 0"/>
@@ -238,3 +113,4 @@
   <!-- <xacro:boris_arm parent="arm_support_link" xyz="0.1 0 ${arm_support_height/2}" rpy="0 0 0"/> -->
   <!-- <xacro:rgb_cam parent="wx200/gripper_bar_link" name="webcam" xyz="-0.078 0.0 0.05" rpy="0 0 0"/> -->
+  <xacro:shark_base/>
 </robot>

File: shark_description/urdf/shark_description.xacro (robot description, xacro)
@@ -90,4 +90,4 @@
     <xacro:wheel prefix="right" reflect="-1" />
   </xacro:macro>
-  <xacro:shark_base/>
+  <!-- <xacro:shark_base/> -->
 </robot>

Commit message: test changes to urdf for gazebo

File: boris_description/urdf/boris.xacro (robot description, xacro)
@@ -1,5 +1,5 @@
 <?xml version="1.0"?>
 <robot xmlns:xacro="http://www.ros.org/wiki/xacro" name="shark-v1">
-  <xacro:include filename="$(find sensors_description)/urdf/hokuyo.xacro" />
+  <!-- <xacro:include filename="$(find sensors_description)/urdf/hokuyo.xacro" /> -->
   <xacro:include filename="$(find sensors_description)/urdf/sick_lms1xx.xacro" />
   <!-- <xacro:include filename="$(find sensors_description)/urdf/realsense_camera.urdf.xacro" /> -->
@@ -223,9 +223,9 @@
     <child link="sick_link" />
   </joint>
-  <joint name="dorso_head" type="fixed">
+  <!-- <joint name="dorso_head" type="fixed">
     <parent link="dorso_link" />
     <child link="head_root" />
     <origin xyz="0 0 ${dorso_height + 0.04}" rpy="0 0 0" />
-  </joint>
+  </joint> -->
   <!-- <xacro:realsense_camera name="camera" parent="dorso_link">
     <origin xyz="${dorso_len/2 + 0.05} 0 ${dorso_height + 0.053}" rpy="0 0 0" />
@@ -233,6 +233,6 @@
   <xacro:dorso parent="base_link" depth="${dorso_len}" width="${dorso_width}" height="${dorso_height}" xyz="${-base_len/2 + (dorso_len/2)} 0 ${base_height/2}" rpy="0 0 0"/>
   <xacro:arm_support parent="dorso_link" width="${arm_support_width}" height="${arm_support_height}" depth="${arm_support_len}" xyz="${dorso_len/2 + arm_support_len/2} 0 ${arm_z_position}" rpy="0 0 0"/>
-  <xacro:sensor_hokuyo parent="base_link" xyz="${base_len/2 + 0.017 + 0.024} 0 ${0.02 - base_height/2}" rpy="3.14 0 0" name="ground"/>
-  <xacro:sensor_hokuyo parent="base_link" xyz="${-base_len/2 - 0.017 - 0.024} 0 ${0.02 - base_height/2}" rpy="3.14 0 3.14" name="back"/>
+  <!-- <xacro:sensor_hokuyo parent="base_link" xyz="${base_len/2 + 0.017 + 0.024} 0 ${0.02 - base_height/2}" rpy="3.14 0 0" name="ground"/>
+  <xacro:sensor_hokuyo parent="base_link" xyz="${-base_len/2 - 0.017 - 0.024} 0 ${0.02 - base_height/2}" rpy="3.14 0 3.14" name="back"/> -->
   <xacro:imu parent="base_link" xyz="-0.01 0 ${0.02 - base_height/2}" rpy="-0.014161 -0.0203861 0" />
   <!-- <xacro:boris_arm parent="arm_support_link" xyz="0.1 0 ${arm_support_height/2}" rpy="0 0 0"/> -->

Commit message: xacro loading in gazebo

File: boris_description/urdf/boris.xacro (robot description, xacro)
@@ -2,5 +2,5 @@
 <robot xmlns:xacro="http://www.ros.org/wiki/xacro" name="shark-v1">
   <!-- <xacro:include filename="$(find sensors_description)/urdf/hokuyo.xacro" /> -->
-  <xacro:include filename="$(find sensors_description)/urdf/sick_lms1xx.xacro" />
+  <!-- <xacro:include filename="$(find sensors_description)/urdf/sick_lms1xx.xacro" /> -->
   <!-- <xacro:include filename="$(find sensors_description)/urdf/realsense_camera.urdf.xacro" /> -->
   <!-- <xacro:include filename="$(find hector_sensors_description)/urdf/realsense_d435_camera.urdf.xacro" /> -->
@@ -10,9 +10,9 @@
   <xacro:property name="base_len" value="0.5" />
   <xacro:property name="base_height" value="0.231" />
-  <xacro:property name="wheel_radius" value="0.0825" />
+  <!-- <xacro:property name="wheel_radius" value="0.0825" />
   <xacro:property name="base_wheel_gap" value="0.05" />
   <xacro:property name="wheel_width" value="0.06" />
   <xacro:property name="wheel_separation" value="0.39" />
-  <xacro:property name="wheel_joint_offset" value="0.0" />
+  <xacro:property name="wheel_joint_offset" value="0.0" /> -->
   <xacro:property name="caster_height" value="0.07" />
   <xacro:property name="dorso_width" value="0.338" />
@@ -90,5 +90,5 @@
     </inertial>
   </xacro:macro>
-  <xacro:macro name="wheel" params="prefix reflect">
+  <!-- <xacro:macro name="wheel" params="prefix reflect">
     <link name="${prefix}_wheel">
       <visual>
@@ -117,5 +117,5 @@
   </xacro:macro>
   <xacro:wheel prefix="left" reflect="1" />
-  <xacro:wheel prefix="right" reflect="-1" />
+  <xacro:wheel prefix="right" reflect="-1" /> -->
   <xacro:macro name="sphere_inertia" params="m r">
     <inertial>
@@ -133,5 +133,5 @@
     </joint>
   </xacro:macro>
-  <xacro:sick_lms1xx />
+  <!-- <xacro:sick_lms1xx /> -->
   <xacro:macro name="dorso" params="parent depth width height xyz rpy">
     <link name="dorso_link">
@@ -218,9 +218,9 @@
     </joint>
   </xacro:macro>
-  <joint name="laser_joint" type="fixed">
+  <!-- <joint name="laser_joint" type="fixed">
     <origin xyz="${base_len/2 + 0.017 + 0.05} 0 ${0.02 + base_height/2}" rpy="0 0 0" />
     <parent link="base_link" />
     <child link="sick_link" />
-  </joint>
+  </joint> -->
   <!-- <joint name="dorso_head" type="fixed">
     <parent link="dorso_link" />
