Commit message: Add caster wheel for gazebo simulation

File: boris_description/urdf/boris.xacro (robot description, xacro)
@@ -7,5 +7,5 @@
   <xacro:include filename="$(find sensors_description)/urdf/realsense_camera.urdf.xacro" />
   <xacro:include filename="$(find boris_head_description)/urdf/boris_head.urdf" />
-  <!-- <xacro:include filename="$(find interbotix_xsarm_descriptions)/urdf/wx200.urdf.xacro" /> -->
+  <xacro:include filename="$(find boris_head_description)/urdf/control.urdf.xacro" />
   <xacro:property name="base_width" value="0.336" />
   <xacro:property name="base_len" value="0.5" />
@@ -47,5 +47,5 @@
     </joint>
   </xacro:macro>
-  <xacro:sick_lms1xx />
+  <xacro:sick_lms1xx robot_namespace="/lms1xx" />
   <xacro:macro name="dorso" params="parent depth width height xyz rpy">
     <link name="dorso_link">
@@ -69,7 +69,6 @@
         <child link="dorso_link"/>
         <origin xyz="${xyz}" rpy="${rpy}"/>
-    </joint>0
+    </joint>
   </xacro:macro>
-    <!--32,5-->
   <xacro:macro name="arm_support" params="parent width height depth xyz rpy">
     <link name="arm_support_link">
@@ -104,6 +103,8 @@
   </joint>
   <xacro:realsense_camera name="camera" parent="dorso_link">
-    <origin xyz="${dorso_len/2 + 0.05} 0 ${dorso_height + 0.053}" rpy="0 0 0" />
+    <origin xyz="${dorso_len/2 + 0.05} 0 ${dorso_height + 0.053}" rpy="0 0 ${3.14/8}" />
   </xacro:realsense_camera>
+  <xacro:realsense_gazebo />
+  <xacro:add_optical_frame name="camera_link" />
   <xacro:dorso parent="base_link" depth="${dorso_len}" width="${dorso_width}" height="${dorso_height}" xyz="${-base_len/2 + (dorso_len/2)} 0 ${base_height/2}" rpy="0 0 0"/>
   <xacro:arm_support parent="dorso_link" width="${arm_support_width}" height="${arm_support_height}" depth="${arm_support_len}" xyz="${dorso_len/2 + arm_support_len/2} 0 ${arm_z_position}" rpy="0 0 0"/>
@@ -111,6 +112,9 @@
   <xacro:sensor_hokuyo parent="base_link" xyz="${-base_len/2 - 0.017 - 0.024} 0 ${0.02 - base_height/2}" rpy="3.14 0 3.14" name="back"/>
   <xacro:imu parent="base_link" xyz="-0.01 0 ${0.02 - base_height/2}" rpy="-0.014161 -0.0203861 0" />
-  <!-- <xacro:boris_arm parent="arm_support_link" xyz="0.1 0 ${arm_support_height/2}" rpy="0 0 0"/> -->
-  <!-- <xacro:rgb_cam parent="wx200/gripper_bar_link" name="webcam" xyz="-0.078 0.0 0.05" rpy="0 0 0"/> -->
-  <xacro:shark_base/>  <!-- isso aq n existe mais, a gente reverteu as mudanças do luis que transformavam aquilo tudo em um macro q n ta aparecendo mais -->
+  <gazebo reference="dorso_link">
+    <material>Gazebo/DarkGray</material>
+  </gazebo>
+  <gazebo reference="arm_support_link">
+    <material>Gazebo/DarkGray</material>
+  </gazebo>
 </robot>

File: sensors_description/urdf/hokuyo.xacro (robot description, xacro)
@@ -4,10 +4,4 @@
   <xacro:macro name="sensor_hokuyo" params="parent xyz rpy name">
     <link name="hokuyo_${name}_link">
-      <!--collision>
-        <origin xyz="0 0 0" rpy="0 0 0"/>
-        <geometry>
-          <box size="0.01 0.01 0.01"/>
-        </geometry>
-      </collision-->
       <visual>
         <origin xyz="0 0 0" rpy="0 0 0"/>
@@ -23,18 +17,15 @@
     </link>
     <joint name="hokuyo_${name}_joint" type="fixed">
-      <!--<axis xyz="0 0 1" />-->
       <origin xyz="${xyz}" rpy="${rpy}"/>
       <parent link="${parent}"/>
       <child link="hokuyo_${name}_link"/>
     </joint>
-    <!-- Hokuyo sensor for simulation -->
-    <xacro:sim_laser_range_finder/>
+    <xacro:sim_laser_range_finder name="${name}"/>
   </xacro:macro>
-  <!-- ULM-30LX Hokuyo Laser Range Finder -->
-  <xacro:macro name="sim_laser_range_finder">
+  <xacro:macro name="sim_laser_range_finder" params="name">
     <gazebo reference="hokuyo_${name}_link">
-      <sensor type="ray" name="head_hokuyo_sensor">
+      <sensor type="gpu_ray" name="${name}_hokuyo_sensor">
         <pose>0 0 0 0 0 0</pose>
-        <visualize>false</visualize>
+        <visualize>true</visualize>
         <update_rate>40</update_rate>
         <ray>
@@ -54,16 +45,14 @@
           <noise>
             <type>gaussian</type>
-            <!-- Noise parameters based on published spec for Hokuyo laser
-               achieving "+-30mm" accuracy at range < 10m.  A mean of 0.0m and
-               stddev of 0.01m will put 99.7% of samples within 0.03m of the true
-               reading. -->
             <mean>0.0</mean>
             <stddev>0.01</stddev>
           </noise>
         </ray>
-        <plugin name="gazebo_ros_head_hokuyo_controller" filename="libgazebo_ros_laser.so">
-          <topicName>scan2</topicName>
-          <frameName>hokuyo_${name}_link</frameName>
-          <robotNamespace>/</robotNamespace>
+        <plugin name="gazebo_ros_${name}_hokuyo_controller" filename="libgazebo_ros_ray_sensor.so">
+          <ros>
+            <remapping>~/out:=/${name}/scan</remapping>
+            <namespace>/${name}</namespace>
+          </ros>
+          <output_type>sensor_msgs/LaserScan</output_type>
         </plugin>
       </sensor>

File: sensors_description/urdf/realsense_camera.urdf.xacro (robot description, xacro)
@@ -2,6 +2,81 @@
 <robot xmlns:xacro="http://www.ros.org/wiki/xacro">
   <xacro:property name="M_PI" value="3.1415926535897931"/>
+  <xacro:macro name="add_optical_frame" params="name">
+		<joint name="${name}_optical_joint" type="fixed">
+			<origin xyz="0 0 0" rpy="0.0 0.0 0.0" />
+			<parent link="${name}" />
+			<child link="${name}_optical_frame"/>
+		</joint>
+		<link name="${name}_optical_frame" />
+	</xacro:macro>
+  <xacro:macro name="realsense_gazebo">
+		<gazebo reference="camera_link_optical_frame">
+			<sensor type="camera" name="realsense">
+				<always_on>true</always_on>
+				<visualize>true</visualize>
+				<update_rate>15</update_rate>
+				<gz_frame_id>camera_link_optical_frame</gz_frame_id>
+				<camera>
+					<optical_frame_id>camera_link_optical_frame</optical_frame_id>
+					<horizontal_fov>1.047</horizontal_fov>
+					<image>
+						<width>640</width>
+						<height>480</height>
+					</image>
+					<depth_camera>
+						<clip>
+							<near>0.1</near>
+							<far>10.0</far>
+						</clip>
+					</depth_camera>
+					<noise>
+						<type>gaussian</type>
+						<mean>0.0</mean>
+						<stddev>0.01</stddev>
+					</noise>
+				</camera>
+                <plugin name="realsense_camera_plugin" filename="libgazebo_ros_camera.so">
+                    <ros>
+                    <remapping>image_raw:=/realsense/image_color/raw</remapping>
+                    <remapping>camera_info:=/realsense/image_color/camera_info</remapping>
+                    <frame_name>camera_link_optical_frame</frame_name>
+                    </ros>
+                </plugin>
+			</sensor>
+            <sensor type="depth" name="realsense_depth">
+				<always_on>true</always_on>
+				<visualize>true</visualize>
+				<update_rate>15</update_rate>
+				<gz_frame_id>camera_link_optical_frame</gz_frame_id>
+				<camera>
+					<optical_frame_id>camera_link_optical_frame</optical_frame_id>
+					<horizontal_fov>1.047</horizontal_fov>
+					<image>
+						<width>640</width>
+						<height>480</height>
+					</image>
+					<depth_camera>
+						<clip>
+							<near>0.1</near>
+							<far>10.0</far>
+						</clip>
+					</depth_camera>
+					<noise>
+						<type>gaussian</type>
+						<mean>0.0</mean>
+						<stddev>0.01</stddev>
+					</noise>
+				</camera>
+                <plugin name="realsense_camera_plugin" filename="libgazebo_ros_camera.so">
+                    <ros>
+                    <remapping>image_raw:=/realsense/image_depth/raw</remapping>
+                    <remapping>camera_info:=/realsense/image_depth/camera_info</remapping>
+                    <frame_name>camera_link_optical_frame</frame_name>
+                    </ros>
+                </plugin>
+			</sensor>
+		</gazebo>
+	</xacro:macro>
   <xacro:macro name="realsense_camera" params="name parent *origin">
-      <!-- @TODO: GABIARRA PRA GIRAR A CAMERA -->
       <link name="head_pan_link_static">
           <inertial>
@@ -131,7 +206,19 @@
           <axis xyz="0 0 0"/>
       </joint>
-      <!-- <xacro:sensor_d435 parent="head_tilt_link" use_nominal_extrinsics="false" add_plug="false" use_mesh="true">
-          <origin xyz="0.06705 0 -0.00425" rpy="0 0 0"/>
-      </xacro:sensor_d435> -->
+      <ros2_control name="head_hardware_interface" type="system">
+    <hardware>
+      <plugin>gazebo_ros2_control/GazeboSystem</plugin>
+    </hardware>
+    <joint name="head_pan_joint">
+      <command_interface name="position">
+      </command_interface>
+      <state_interface name="position"/>
+    </joint>
+    <joint name="head_tilt_joint">
+      <command_interface name="position">
+      </command_interface>
+      <state_interface name="position"/>
+    </joint>
+  </ros2_control>
   </xacro:macro>
 </robot>

File: sensors_description/urdf/rgb_cam.xacro (robot description, xacro)
@@ -1,4 +1,48 @@
 <?xml version="1.0"?>
 <robot xmlns:xacro="http://www.ros.org/wiki/xacro" name="rgb_cam">
+<xacro:macro name="add_optical_frame_rgb_cam" params="name">
+		<joint name="${name}_optical_joint" type="fixed">
+			<origin xyz="0 0 0" rpy="0.0 0.0 0.0" />
+			<parent link="${name}" />
+			<child link="${name}_optical_frame"/>
+		</joint>
+		<link name="${name}_optical_frame" />
+	</xacro:macro>
+  <xacro:macro name="rgb_cam_gazebo">
+		<gazebo reference="webcam_lens_link_optical_frame">
+			<sensor type="camera" name="rgb_cam">
+				<always_on>true</always_on>
+				<visualize>true</visualize>
+				<update_rate>15</update_rate>
+				<gz_frame_id>webcam_lens_link_optical_frame</gz_frame_id>
+				<camera>
+					<optical_frame_id>webcam_lens_link_optical_frame</optical_frame_id>
+					<horizontal_fov>1.047</horizontal_fov>
+					<image>
+						<width>640</width>
+						<height>480</height>
+					</image>
+					<depth_camera>
+						<clip>
+							<near>0.1</near>
+							<far>10.0</far>
+						</clip>
+					</depth_camera>
+					<noise>
+						<type>gaussian</type>
+						<mean>0.0</mean>
+						<stddev>0.01</stddev>
+					</noise>
+				</camera>
+                <plugin name="rgb_cam_camera_plugin" filename="libgazebo_ros_camera.so">
+                    <ros>
+                    <remapping>image_raw:=/rgb_cam/image_color/raw</remapping>
+                    <remapping>camera_info:=/rgb_cam/image_color/camera_info</remapping>
+                    <frame_name>webcam_lens_link_optical_frame</frame_name>
+                    </ros>
+                </plugin>
+			</sensor>
+		</gazebo>
+	</xacro:macro>
     <xacro:macro name="rgb_cam" params="parent name xyz rpy">
         <link name="${name}_link">

File: sensors_description/urdf/sick_lms1xx.xacro (robot description, xacro)
@@ -1,28 +1,3 @@
 <?xml version="1.0"?>
-<!--
-Copyright (c) 2013, Goncalo Cabrita, ISR University of Coimbra
-Copyright (c) 2014, 2015 Clearpath Robotics
-All rights reserved.
-Redistribution and use in source and binary forms, with or without
-modification, are permitted provided that the following conditions are met:
-    * Redistributions of source code must retain the above copyright
-      notice, this list of conditions and the following disclaimer.
-    * Redistributions in binary form must reproduce the above copyright
-      notice, this list of conditions and the following disclaimer in the
-      documentation and/or other materials provided with the distribution.
-    * Neither the name of Clearpath Robotics nor the
-      names of its contributors may be used to endorse or promote products
-      derived from this software without specific prior written permission.
-THIS SOFTWARE IS PROVIDED BY THE COPYRIGHT HOLDERS AND CONTRIBUTORS "AS IS" AND
-ANY EXPRESS OR IMPLIED WARRANTIES, INCLUDING, BUT NOT LIMITED TO, THE IMPLIED
-WARRANTIES OF MERCHANTABILITY AND FITNESS FOR A PARTICULAR PURPOSE ARE
-DISCLAIMED. IN NO EVENT SHALL THE COPYRIGHT HOLDERS BE LIABLE FOR ANY
-DIRECT, INDIRECT, INCIDENTAL, SPECIAL, EXEMPLARY, OR CONSEQUENTIAL DAMAGES
-(INCLUDING, BUT NOT LIMITED TO, PROCUREMENT OF SUBSTITUTE GOODS OR SERVICES;
-LOSS OF USE, DATA, OR PROFITS; OR BUSINESS INTERRUPTION) HOWEVER CAUSED AND
-ON ANY THEORY OF LIABILITY, WHETHER IN CONTRACT, STRICT LIABILITY, OR TORT
-(INCLUDING NEGLIGENCE OR OTHERWISE) ARISING IN ANY WAY OUT OF THE USE OF THIS
-SOFTWARE, EVEN IF ADVISED OF THE POSSIBILITY OF SUCH DAMAGE.
--->
 <robot xmlns:xacro="http://www.ros.org/wiki/xacro">
   <xacro:macro name="sick_lms1xx" params="frame:=sick_link topic:=scan sample_size:=720 update_rate:=50
@@ -39,19 +14,12 @@
         <origin xyz="0 0 0" rpy="0 0 0" />
         <geometry>
-          <!-- Origin of this mesh is the focal point of the LIDAR. -->
-          <mesh filename="package://lms1xx/meshes/sick-lms1xx.dae" />
+          <mesh filename="package://sensors_description/meshes/sick-lms1xx.dae" />
         </geometry>
       </visual>
-      <!--collision>
-        <origin xyz="0 0 -0.05" rpy="0 0 0" />
-        <geometry>
-          <box size="0.105 0.1 0.1" />
-        </geometry>
-      </collision-->
     </link>
     <gazebo reference="${frame}">
-      <sensor type="ray" name="${frame}">
+      <sensor type="gpu_ray" name="${frame}">
         <pose>0 0 0 0 0 0</pose>
-        <visualize>false</visualize>
+        <visualize>true</visualize>
         <update_rate>${update_rate}</update_rate>
         <ray>
@@ -75,8 +43,10 @@
           </noise>
         </ray>
-        <plugin name="gazebo_ros_laser" filename="libgazebo_ros_laser.so">
-          <topicName>${topic}</topicName>
-          <frameName>${frame}</frameName>
-          <robotNamespace>${robot_namespace}</robotNamespace>
+        <plugin name="gazebo_ros_laser" filename="libgazebo_ros_ray_sensor.so">
+          <ros>
+            <namespace>${robot_namespace}</namespace>
+            <remapping>~/out:=${topic}</remapping>
+          </ros>
+          <output_type>sensor_msgs/LaserScan</output_type>
         </plugin>
       </sensor>

File: sensors_description/urdf/velodyne.xacro (robot description, xacro)
@@ -1,5 +1,4 @@
 <?xml version="1.0"?>
 <robot xmlns:xacro="http://www.ros.org/wiki/xacro" name="velodyne">
-  <!-- Inclui o arquivo URDF do Velodyne VLP-16 -->
   <xacro:include filename="$(find velodyne_description)/urdf/VLP-16.urdf.xacro"/>
 </robot>

File: shark_description/urdf/shark.xacro (robot description, xacro)
@@ -1,9 +1,12 @@
 <?xml version="1.0"?>
-<!-- Basic differential drive mobile base -->
 <robot xmlns:xacro="http://www.ros.org/wiki/xacro" name="shark">
+  <xacro:property name="hardware_type" value="gz_classic" />
   <xacro:include filename="$(find shark_description)/urdf/shark_description.xacro" />
-  <!-- Import Rviz colors -->
   <xacro:include filename="$(find shark_description)/urdf/shark_materials.xacro" />
-  <!-- Import diffbot ros2_control description -->
-  <xacro:include filename="$(find shark_description)/ros2_control/shark_ros2_control.xacro" />
+  <xacro:if value="${hardware_type == 'actual'}">
+    <xacro:include filename="$(find shark_description)/ros2_control/shark_ros2_control.xacro" />
+  </xacro:if>
+  <xacro:if value="${hardware_type == 'gz_classic'}">
+    <xacro:include filename="$(find shark_description)/urdf/shark_v1_gazebo_plugins.xacro" />
+  </xacro:if>
 </robot>

File: shark_description/urdf/shark_description.xacro (robot description, xacro)
@@ -10,4 +10,6 @@
   <xacro:property name="wheel_joint_offset" value="0.0" />
   <xacro:property name="caster_height" value="0.07" />
+  <xacro:property name="caster_wheel_joint_offset" value="0.0" />
+  <xacro:property name="caster_wheel_radius" value="0.02" />
   <xacro:macro name="box_inertia" params="m w h d">
     <inertial>
@@ -68,5 +70,5 @@
       <xacro:cylinder_inertia m="10" r="${wheel_radius}" h="0.05"/>
     </link>
-    <joint name="${prefix}_wheel" type="continuous">
+    <joint name="${prefix}_wheel_joint" type="continuous">
       <axis xyz="0 1 0" rpy="0 0 0" />
       <parent link="base_link"/>
@@ -83,5 +85,5 @@
     </inertial>
   </xacro:macro>
-   <!-- <link name="caster_wheel">
+   <link name="caster_wheel">
      <visual>
        <material name="darkgray"/>
@@ -103,5 +105,5 @@
     <parent link="base_link"/>
     <child link="caster_wheel"/>
-    <origin xyz="${caster_wheel_joint_offset} 0 -${0.06+caster_wheel_radius}" rpy="0 0 0"/>
-  </joint> -->
+    <origin xyz="${(base_len/2) - caster_wheel_joint_offset} 0 ${(caster_wheel_radius - caster_height) - base_height/2}" rpy="0 0 0"/>
+  </joint>
 </robot>

File: shark_description/urdf/shark_materials.xacro (robot description, xacro)
@@ -1,7 +1,3 @@
 <?xml version="1.0"?>
-<!--
-Copied from ROS1 example:
-https://github.com/ros-simulation/gazebo_ros_demos/blob/kinetic-devel/rrbot_description/urdf/materials.xacro
--->
 <robot>
   <material name="blue">

File: shark_description/urdf/shark_v1_gazebo_plugins.xacro (robot description, xacro)
@@ -1,18 +1,19 @@
 <?xml version="1.0"?>
 <robot>
-<!--Gazebo Differential Drive Plugin-->
   <gazebo>
         <plugin name='diff_drive' filename='libgazebo_ros_diff_drive.so'>
-            <!-- Wheel Information -->
+            <ros>
+                <namespace>/</namespace>
+            </ros>
             <left_joint>left_wheel_joint</left_joint>
             <right_joint>right_wheel_joint</right_joint>
             <wheel_separation>${wheel_separation}</wheel_separation>
             <wheel_diameter>${wheel_radius}</wheel_diameter>
-            <!-- Limits -->
             <max_wheel_torque>200</max_wheel_torque>
             <max_wheel_acceleration>10.0</max_wheel_acceleration>
-            <!-- Output -->
             <odometry_frame>odom</odometry_frame>
-            <robot_base_frame>base_link</robot_base_frame>
+            <robot_base_frame>base_footprint</robot_base_frame>
+            <command_topic>/cmd_vel</command_topic>
+            <odometry_topic>/odom</odometry_topic>
             <publish_odom>true</publish_odom>
             <publish_odom_tf>true</publish_odom_tf>
@@ -20,3 +21,26 @@
         </plugin>
     </gazebo>
+    <gazebo>
+        <link name="base_link">
+            <sensor name="imu" type="imu">
+                <always_on>true</always_on>
+                <update_rate>30</update_rate>
+                <plugin name="imu_plugin" filename="libgazebo_ros_imu_sensor.so">
+                <ros>
+                    <namespace>/bno055</namespace>
+                    <remapping>~/out:=imu</remapping>
+                </ros>
+                </plugin>
+            </sensor>
+        </link>
+    </gazebo>
+    <gazebo reference="base_link">
+      <material>Gazebo/DarkGray</material>
+    </gazebo>
+    <gazebo reference="left_wheel">
+      <material>Gazebo/Black</material>
+    </gazebo>
+    <gazebo reference="right_wheel">
+      <material>Gazebo/Black</material>
+    </gazebo>
 </robot>
