Commit message: changes to xacros

File: boris_description/urdf/boris.xacro (robot description, xacro)
@@ -4,4 +4,7 @@
   <xacro:include filename="$(find sensors_description)/urdf/sick_lms1xx.xacro" />
   <xacro:include filename="$(find sensors_description)/urdf/rgb_cam.xacro" />
+  <xacro:include filename="$(find sensors_description)/urdf/camera_turret.xacro" />
+  <xacro:include filename="$(find hector_models)/urdf/orbbec_astra2.xacro" />
+  <xacro:include filename="$(find hector_models)/gazebo/orbbec_astra2.gazebo.xacro" />
   <xacro:include filename="$(find shark_description)/urdf/shark.xacro" />
   <xacro:include filename="$(find sensors_description)/urdf/realsense_camera.urdf.xacro" />
@@ -102,9 +105,12 @@
     <origin xyz="0 0 ${dorso_height + 0.04}" rpy="0 0 0" />
   </joint>
-  <xacro:realsense_camera name="camera" parent="dorso_link">
+  <xacro:camera_turret parent="dorso_link" name="camera_turret">
     <origin xyz="${dorso_len/2 + 0.05} 0 ${dorso_height + 0.053}" rpy="0 0 ${3.14/8}" />
-  </xacro:realsense_camera>
-  <xacro:realsense_gazebo />
-  <xacro:add_optical_frame name="camera_link" />
+  </xacro:camera_turret>
+  <xacro:orbbec_astra2 name="top_camera">
+    <parent link="camera_turret_tilt_link"/>
+    <origin rpy="0 0 0" xyz="0.06705 0 -0.00425"/>
+  </xacro:orbbec_astra2>
+  <xacro:orbbec_astra2_gazebo name="top_camera" semantic_segmentation="false"/>
   <xacro:dorso parent="base_link" depth="${dorso_len}" width="${dorso_width}" height="${dorso_height}" xyz="${-base_len/2 + (dorso_len/2)} 0 ${base_height/2}" rpy="0 0 0"/>
   <xacro:arm_support parent="dorso_link" width="${arm_support_width}" height="${arm_support_height}" depth="${arm_support_len}" xyz="${dorso_len/2 + arm_support_len/2} 0 ${arm_z_position}" rpy="0 0 0"/>

File: boris_description/urdf/boris_arm.xacro (robot description, xacro)
@@ -1,4 +1,6 @@
 <?xml version="1.0"?>
 <robot xmlns:xacro="http://www.ros.org/wiki/xacro" name="shark-v1">
+    <xacro:include filename="$(find hector_models)/urdf/orbbec_astra2.xacro" />
+    <xacro:include filename="$(find hector_models)/gazebo/orbbec_astra2.gazebo.xacro" />
     <xacro:include filename="$(find sensors_description)/urdf/rgb_cam.xacro" />
     <xacro:arg name="robot_name" default="${robot_model}"/>
@@ -9,6 +11,8 @@
         <origin xyz="0.1 0 ${arm_support_height/2}" rpy="0 0 0" />
     </joint>
-    <xacro:rgb_cam parent="wx200/gripper_bar_link" name="webcam" xyz="-0.078 0.0 0.05" rpy="0 0 0"/>
-    <xacro:rgb_cam_gazebo />
-    <xacro:add_optical_frame_rgb_cam name="webcam_lens_link" />
+    <xacro:orbbec_astra2 name="wrist_camera">
+        <parent link="wx200/gripper_bar_link" />
+        <origin xyz="-0.078 0.0 0.05" rpy="0 0 0"/>
+    </xacro:orbbec_astra2>
+    <xacro:orbbec_astra2_gazebo name="wrist_camera" semantic_segmentation="false"/>
 </robot>

File: sensors_description/urdf/hokuyo.xacro (robot description, xacro)
@@ -54,4 +54,5 @@
             <namespace>/${name}</namespace>
           </ros>
+					<frame_name>hokuyo_${name}_link</frame_name>
           <output_type>sensor_msgs/LaserScan</output_type>
         </plugin>

File: sensors_description/urdf/sick_lms1xx.xacro (robot description, xacro)
@@ -49,4 +49,5 @@
           </ros>
           <output_type>sensor_msgs/LaserScan</output_type>
+					<frame_name>${frame}</frame_name>
         </plugin>
       </sensor>

File: shark_description/urdf/shark_description.xacro (robot description, xacro)
@@ -19,12 +19,4 @@
   </xacro:macro>
   <link name="base_footprint">
-    <xacro:box_inertia m="8" w="0.001" h="0.001" d="0.001"/>
-    <visual>
-      <origin xyz="0 0 0" rpy="0 0 0" />
-      <material name="white"/>
-        <geometry>
-            <box size="0.001 0.001 0.001" />
-        </geometry>
-    </visual>
   </link>
   <link name="base_link">

File: shark_description/urdf/shark_v1_gazebo_plugins.xacro (robot description, xacro)
@@ -10,10 +10,9 @@
             <wheel_separation>${wheel_separation}</wheel_separation>
             <wheel_diameter>${wheel_radius}</wheel_diameter>
+            <update_rate>500</update_rate>
             <max_wheel_torque>200</max_wheel_torque>
             <max_wheel_acceleration>10.0</max_wheel_acceleration>
             <odometry_frame>odom</odometry_frame>
             <robot_base_frame>base_footprint</robot_base_frame>
-            <command_topic>/cmd_vel</command_topic>
-            <odometry_topic>/odom</odometry_topic>
             <publish_odom>true</publish_odom>
             <publish_odom_tf>true</publish_odom_tf>

Commit message: Changes to make it possible to simulate Boris on Ignition.

File: boris_description/urdf/boris.xacro (robot description, xacro)
@@ -110,7 +110,7 @@
   <xacro:orbbec_astra2 name="top_camera">
     <parent link="camera_turret_tilt_link"/>
-    <origin rpy="0 0 0" xyz="0.06705 0 -0.00425"/>
+    <origin rpy="0 0 -${M_PI/6}" xyz="0.06705 0 -0.00425"/>
   </xacro:orbbec_astra2>
-  <xacro:orbbec_astra2_gazebo name="top_camera" semantic_segmentation="false"/>
+  <xacro:orbbec_astra2_gazebo name="top_camera"/>
   <xacro:dorso parent="base_link" depth="${dorso_len}" width="${dorso_width}" height="${dorso_height}" xyz="${-base_len/2 + (dorso_len/2)} 0 ${base_height/2}" rpy="0 0 0"/>
   <xacro:arm_support parent="dorso_link" width="${arm_support_width}" height="${arm_support_height}" depth="${arm_support_len}" xyz="${dorso_len/2 + arm_support_len/2} 0 ${arm_z_position}" rpy="0 0 0"/>

File: boris_description/urdf/boris_arm.xacro (robot description, xacro)
@@ -15,4 +15,4 @@
         <origin xyz="-0.078 0.0 0.05" rpy="0 0 0"/>
     </xacro:orbbec_astra2>
-    <xacro:orbbec_astra2_gazebo name="wrist_camera" semantic_segmentation="false"/>
+    <xacro:orbbec_astra2_gazebo name="wrist_camera"/>
 </robot>

File: boris_description/urdf/boris_full.xacro (robot description, xacro)
@@ -3,4 +3,5 @@
     <xacro:property name="robot_model" default="wx200"/>
     <xacro:include filename="$(find boris_description)/urdf/boris_arm.xacro" />
+    <xacro:include filename="$(find boris_description)/urdf/boris_ros2_control.xacro" />
     <xacro:include filename="$(find interbotix_xsarm_descriptions)/urdf/wx200.urdf.xacro" />
 </robot>

File: sensors_description/urdf/camera_turret.xacro (robot description, xacro)
@@ -30,4 +30,5 @@
           <child link="${name}_pan_link"/>
           <axis xyz="0 0 1"/>
+          <dynamics damping="100.0" friction="100.0"/>
           <limit effort="1" lower="-1.57" upper="1.57" velocity="1"/>
       </joint>
@@ -59,4 +60,5 @@
           <child link="${name}_tilt_link"/>
           <axis xyz="0 1 0"/>
+          <dynamics damping="100.0" friction="100.0"/>
           <limit effort="1" lower="-1.57" upper="1.57" velocity="1"/>
         </joint>

File: sensors_description/urdf/hokuyo.xacro (robot description, xacro)
@@ -29,4 +29,6 @@
         <visualize>true</visualize>
         <update_rate>40</update_rate>
+        <topic>/${name}/scan</topic>
+        <gz_frame_id>hokuyo_${name}_link</gz_frame_id>
         <ray>
           <scan>

File: sensors_description/urdf/sick_lms1xx.xacro (robot description, xacro)
@@ -21,4 +21,6 @@
       <sensor type="gpu_ray" name="${frame}">
         <pose>0 0 0 0 0 0</pose>
+        <topic>/${robot_namespace}/${topic}</topic>
+        <gz_frame_id>${frame}</gz_frame_id>
         <visualize>true</visualize>
         <update_rate>${update_rate}</update_rate>

File: shark_description/urdf/shark_v1_gazebo_plugins.xacro (robot description, xacro)
@@ -21,16 +21,35 @@
     </gazebo>
     <gazebo>
-        <link name="base_link">
+        <plugin filename="gz-sim-diff-drive-system" name="gz::sim::systems::DiffDrive">
+            <odom_publisher_frequency>50</odom_publisher_frequency>
+            <left_joint>left_wheel_joint</left_joint>
+            <right_joint>right_wheel_joint</right_joint>
+            <wheel_separation>${wheel_separation}</wheel_separation>
+            <wheel_diameter>${wheel_radius}</wheel_diameter>
+            <max_wheel_torque>200</max_wheel_torque>
+            <max_linear_acceleration>10.0</max_linear_acceleration>
+            <topic>cmd_vel</topic>
+            <publish_odom>true</publish_odom>
+            <publish_odom_tf>true</publish_odom_tf>
+            <publish_wheel_tf>true</publish_wheel_tf>
+            <odom_topic>odom</odom_topic>
+            <frame_id>odom</frame_id>
+            <child_frame_id>base_footprint</child_frame_id>
+            <tf_topic>/tf</tf_topic>
+        </plugin>
+    </gazebo>
+    <gazebo>
+        <plugin filename="gz-sim-joint-state-publisher-system" name="gz::sim::systems::JointStatePublisher">
+            <update_rate>50</update_rate>
+            <joint_name>left_wheel_joint</joint_name>
+            <joint_name>right_wheel_joint</joint_name>
+        </plugin>
+    </gazebo>
+    <gazebo reference="base_link">
             <sensor name="imu" type="imu">
                 <always_on>true</always_on>
                 <update_rate>30</update_rate>
-                <plugin name="imu_plugin" filename="libgazebo_ros_imu_sensor.so">
-                <ros>
-                    <namespace>/bno055</namespace>
-                    <remapping>~/out:=imu</remapping>
-                </ros>
-                </plugin>
+                <topic>imu</topic>
             </sensor>
-        </link>
     </gazebo>
     <gazebo reference="base_link">

Commit message: ros-gz-bridge not working

File: boris_description/urdf/boris.xacro (robot description, xacro)
@@ -1,7 +1,11 @@
 <?xml version="1.0"?>
 <robot xmlns:xacro="http://www.ros.org/wiki/xacro" name="shark-v1">
+  <!-- Include xacro utilities for functions like optenv -->
+  <!-- Define environment variable properties before including files that use them -->
+  <xacro:property name="ign_gazebo_resource_path" value="$(optenv IGN_GAZEBO_RESOURCE_PATH)" />
+  <xacro:property name="ign_gazebo_resource_path_set" value="${ign_gazebo_resource_path != ''}" />
   <xacro:include filename="$(find shark_description)/urdf/shark.xacro" />
   <xacro:include filename="$(find sensors_description)/urdf/hokuyo.xacro" />
-  <xacro:include filename="/home/stihl/fbot_ws/src/sick_scan_xd/urdf/sick_lms1xx.urdf.xacro" />
+  <!-- <xacro:include filename="/home/stihl/fbot_ws/src/sick_scan_xd/urdf/sick_lms1xx.urdf.xacro" /> -->
   <xacro:include filename="$(find sensors_description)/urdf/rgb_cam.xacro" />
   <xacro:include filename="$(find sensors_description)/urdf/realsense_camera.xacro" />
@@ -48,5 +52,5 @@
     </joint>
   </xacro:macro>
-  <xacro:sick_lms_1xx name="sick" ros_topic="/scan" />
+  <!-- <xacro:sick_lms_1xx name="sick" ros_topic="/scan" /> -->
   <xacro:macro name="dorso" params="parent depth width height xyz rpy">
     <link name="dorso_link">
@@ -94,4 +98,24 @@
     </joint>
   </xacro:macro>
+  <material name="gray">
+    <color rgba="0.5 0.5 0.5 1.0"/>
+  </material>
+  <link name="sick_mount_link">
+    <visual>
+      <geometry>
+        <box size="0.1 0.1 0.1" />
+      </geometry>
+      <material name="gray" />
+    </visual>
+    <collision>
+      <geometry>
+        <box size="0.1 0.1 0.1" />
+      </geometry>
+    </collision>
+    <inertial>
+      <mass value="0.1" />
+      <inertia ixx="0.001" ixy="0.0" ixz="0.0" iyy="0.001" iyz="0.0" izz="0.001" />
+    </inertial>
+  </link>
   <joint name="laser_joint" type="fixed">
     <origin xyz="${base_len/2 + 0.017 + 0.05} 0 ${0.02 + base_height/2}" rpy="0 0 0" />
@@ -109,5 +133,5 @@
     <child link="wx200/base_link"/>
   </joint> -->
-  <xacro:realsense_camera name="camera" parent="dorso_link" xyz="${dorso_len/2 + 0.05} 0 ${dorso_height + 0.053}" rpy="0 0 0"/>
+  <xacro:shark_base/>
   <xacro:dorso parent="base_link" depth="${dorso_len}" width="${dorso_width}" height="${dorso_height}" xyz="${-base_len/2 + (dorso_len/2)} 0 ${base_height/2}" rpy="0 0 0"/>
   <xacro:arm_support parent="dorso_link" width="${arm_support_width}" height="${arm_support_height}" depth="${arm_support_len}" xyz="${dorso_len/2 + arm_support_len/2} 0 ${arm_z_position}" rpy="0 0 0"/>
@@ -115,6 +139,17 @@
   <xacro:sensor_hokuyo parent="base_link" xyz="${-base_len/2 - 0.017 - 0.024} 0 ${0.02 - base_height/2}" rpy="3.14 0 3.14" name="back"/>
   <xacro:imu parent="base_link" xyz="-0.01 0 ${0.02 - base_height/2}" rpy="-0.014161 -0.0203861 0" />
-  <!-- <xacro:boris_arm parent="arm_support_link" xyz="0.1 0 ${arm_support_height/2}" rpy="0 0 0"/> -->
-  <!-- <xacro:rgb_cam parent="wx200/gripper_bar_link" name="webcam" xyz="-0.078 0.0 0.05" rpy="0 0 0"/> -->
-  <xacro:shark_base/>  <!-- isso aq n existe mais, a gente reverteu as mudanças do luis que transformavam aquilo tudo em um macro q n ta aparecendo mais -->
+  <xacro:realsense_camera name="camera" parent="dorso_link" xyz="${dorso_len/2 + 0.05} 0 ${dorso_height + 0.053}" rpy="0 0 0"/>
+  <!-- Comment out this joint until the WX200 arm is properly included -->
+  <!--
+  <joint name="arm_support_base" type="fixed">
+    <parent link="arm_support_link"/>
+    <child link="wx200/base_link"/>
+    <origin rpy="0 0 0" xyz="0.1 0 0.0235"/>
+  </joint>
+  -->
+  <gazebo>
+    <plugin filename="libgazebo_ros2_control.so" name="gazebo_ros2_control">
+      <parameters>/home/guilherme/fbot_ws/src/fbot_simulation/config/controllers.yaml</parameters>
+    </plugin>
+  </gazebo>
 </robot>

File: sensors_description/urdf/hokuyo.xacro (robot description, xacro)
@@ -13,4 +13,5 @@
         <origin xyz="0 0 0" rpy="0 0 0"/>
         <geometry>
+          <!-- Always use package:// format which is more reliable -->
           <mesh filename="package://sensors_description/meshes/hokuyo.dae"/>
         </geometry>
@@ -34,5 +35,5 @@
   <xacro:macro name="sim_laser_range_finder">
     <gazebo reference="hokuyo_${name}_link">
-      <sensor type="ray" name="head_hokuyo_sensor">
+      <sensor type="ray" name="${name}_hokuyo_sensor">
         <pose>0 0 0 0 0 0</pose>
         <visualize>false</visualize>

File: sensors_description/urdf/realsense_camera.xacro (robot description, xacro)
@@ -3,5 +3,4 @@
   <xacro:property name="M_PI" value="3.1415926535897931"/>
   <xacro:macro name="realsense_camera" params="name parent xyz rpy">
-      <!-- @TODO: GABIARRA PRA GIRAR A CAMERA -->
       <link name="head_pan_link_static">
           <inertial>
@@ -10,4 +9,19 @@
               <inertia ixx="1.32243845065555E-05" ixy="5.07660179129181E-13" ixz="1.067515220067E-20" iyy="7.13386116649085E-06" iyz="-1.32882457845217E-20" izz="7.83291781352837E-06"/>
           </inertial>
+          <visual>
+              <origin rpy="0 0 0" xyz="0 0 0"/>
+              <geometry>
+                  <mesh filename="package://sensors_description/meshes/tilt_link.STL"/>
+              </geometry>
+              <material name="">
+                  <color rgba="0.250980392156863 0.250980392156863 0.250980392156863 1"/>
+              </material>
+          </visual>
+          <collision>
+              <origin rpy="0 0 0" xyz="0 0 0"/>
+              <geometry>
+                  <mesh filename="package://sensors_description/meshes/tilt_link.STL"/>
+              </geometry>
+          </collision>
       </link>
       <link name="head_pan_link">

File: sensors_description/urdf/sick_lms1xx.xacro (robot description, xacro)
@@ -75,9 +75,9 @@
           </noise>
         </ray>
-        <plugin name="gazebo_ros_laser" filename="libgazebo_ros_laser.so">
-          <topicName>${topic}</topicName>
-          <frameName>${frame}</frameName>
-          <robotNamespace>${robot_namespace}</robotNamespace>
-        </plugin>
+        <!-- Comment out the plugin if not required -->
+        <!-- <plugin name="gazebo_ros_laser" filename="libgazebo_ros_laser.so"> -->
+        <!--   <topicName>${topic}</topicName> -->
+        <!--   <frameName>${frame}</frameName> -->
+        <!-- </plugin> -->
       </sensor>
     </gazebo>

File: shark_description/urdf/shark_description.xacro (robot description, xacro)
@@ -23,7 +23,7 @@
   </xacro:macro>
   <xacro:macro name="wheel" params="prefix reflect">
-    <link name="${prefix}_wheel">
+    <link name="${prefix}_wheel_link">
       <visual>
-	      <material name="darkgray"/>
+        <material name="darkgray"/>
         <origin xyz="0 0 0" rpy="${pi/2} 0 0"/>
         <geometry>
@@ -39,8 +39,8 @@
       <xacro:cylinder_inertia m="10" r="${wheel_radius}" h="0.05"/>
     </link>
-    <joint name="${prefix}_wheel" type="continuous">
+    <joint name="${prefix}_wheel_joint" type="continuous">
       <axis xyz="0 1 0" rpy="0 0 0" />
       <parent link="base_link"/>
-      <child link="${prefix}_wheel"/>
+      <child link="${prefix}_wheel_link"/>
       <origin xyz="${wheel_joint_offset} ${((base_width/2)+base_wheel_gap)*reflect} ${(wheel_radius - caster_height) - base_height/2}" rpy="0 0 0"/>
     </joint>

File: shark_description/urdf/shark_v1_gazebo_plugins.xacro (robot description, xacro)
@@ -1,22 +1,22 @@
 <?xml version="1.0"?>
 <robot>
-<!--Gazebo Differential Drive Plugin-->
+  <!-- Gazebo Differential Drive Plugin -->
   <gazebo>
-        <plugin name='diff_drive' filename='libgazebo_ros_diff_drive.so'>
-            <!-- Wheel Information -->
-            <left_joint>left_wheel_joint</left_joint>
-            <right_joint>right_wheel_joint</right_joint>
-            <wheel_separation>${wheel_separation}</wheel_separation>
-            <wheel_diameter>${wheel_radius}</wheel_diameter>
-            <!-- Limits -->
-            <max_wheel_torque>200</max_wheel_torque>
-            <max_wheel_acceleration>10.0</max_wheel_acceleration>
-            <!-- Output -->
-            <odometry_frame>odom</odometry_frame>
-            <robot_base_frame>base_link</robot_base_frame>
-            <publish_odom>true</publish_odom>
-            <publish_odom_tf>true</publish_odom_tf>
-            <publish_wheel_tf>true</publish_wheel_tf>
-        </plugin>
-    </gazebo>
+    <plugin name="diff_drive" filename="libgazebo_ros_diff_drive.so">
+      <!-- Wheel Information -->
+      <left_joint>left_wheel_joint</left_joint>
+      <right_joint>right_wheel_joint</right_joint>
+      <wheel_separation>${wheel_separation}</wheel_separation>
+      <wheel_diameter>${wheel_radius}</wheel_diameter>
+      <!-- Limits -->
+      <max_wheel_torque>200</max_wheel_torque>
+      <max_wheel_acceleration>10.0</max_wheel_acceleration>
+      <!-- Output -->
+      <odometry_frame>odom</odometry_frame>
+      <robot_base_frame>base_link</robot_base_frame>
+      <publish_odom>true</publish_odom>
+      <publish_odom_tf>true</publish_odom_tf>
+      <publish_wheel_tf>true</publish_wheel_tf>
+    </plugin>
+  </gazebo>
 </robot>
