Commit message: Add urdf files required for simulation.

File: boris_description/urdf/boris_ros2_control.xacro (robot description, xacro)
@@ -11,4 +11,5 @@
             </command_interface>
             <state_interface name="position"/>
+            <state_interface name="velocity"/>
         </joint>
         <joint name="shoulder">
@@ -17,7 +18,7 @@
                 <param name="max">6.28</param>
             </command_interface>
-        <state_interface name="position">
-            <param name="initial_value">-1.570</param>
-        </state_interface>
+            <state_interface name="position">
+            </state_interface>
+            <state_interface name="velocity"/>
         </joint>
         <joint name="elbow">
@@ -26,5 +27,6 @@
                 <param name="max">6.28</param>
             </command_interface>
-        <state_interface name="position"/>
+            <state_interface name="position"/>
+            <state_interface name="velocity"/>
         </joint>
         <joint name="wrist_angle">
@@ -33,5 +35,6 @@
                 <param name="max">6.28</param>
             </command_interface>
-        <state_interface name="position"/>
+            <state_interface name="position"/>
+            <state_interface name="velocity"/>
         </joint>
         <joint name="wrist_rotate">
@@ -41,18 +44,151 @@
             </command_interface>
             <state_interface name="position"/>
+            <state_interface name="velocity"/>
         </joint>
         <joint name="left_finger">
             <command_interface name="position">
                 <param name="min">-0.1</param>
-                <param name="max">0.0</param>
-            </command_interface>
-            <state_interface name="position"/>
+                <param name="max">0.1</param>
+            </command_interface>
+            <state_interface name="position"/>
+            <state_interface name="velocity"/>
         </joint>
         <joint name="right_finger">
                 <command_interface name="position">
-                <param name="min">0.0</param>
+                <param name="min">-0.1</param>
                 <param name="max">0.1</param>
                 </command_interface>
                 <state_interface name="position"/>
+                <state_interface name="velocity"/>
+        </joint>
+        <joint name="caster_wheel_joint">
+            <state_interface name="velocity"/>
+            <state_interface name="position"/>
+        </joint>
+        <joint name="gripper">
+            <command_interface name="position">
+                <param name="min">-6.28</param>
+                <param name="max">6.28</param>
+            </command_interface>
+            <state_interface name="position"/>
+        </joint>
+        <joint name="camera_turret_pan_joint">
+            <command_interface name="position">
+                <param name="min">-6.28</param>
+                <param name="max">6.28</param>
+            </command_interface>
+            <state_interface name="position"/>
+        </joint>
+        <joint name="camera_turret_tilt_joint">
+            <command_interface name="position">
+                <param name="min">-6.28</param>
+                <param name="max">6.28</param>
+            </command_interface>
+            <state_interface name="position"/>
+        </joint>
+        <joint name="horizontal_neck_joint">
+            <command_interface name="position">
+                <param name="min">-6.28</param>
+                <param name="max">6.28</param>
+            </command_interface>
+            <state_interface name="position"/>
+        </joint>
+        <joint name="vertical_neck_joint">
+            <command_interface name="position">
+                <param name="min">-6.28</param>
+                <param name="max">6.28</param>
+            </command_interface>
+            <state_interface name="position"/>
+        </joint>
+        <joint name="jaw_joint">
+            <command_interface name="position">
+                <param name="min">-6.28</param>
+                <param name="max">6.28</param>
+            </command_interface>
+            <state_interface name="position"/>
+        </joint>
+        <joint name="left_eye_horizontal_joint">
+            <command_interface name="position">
+                <param name="min">-6.28</param>
+                <param name="max">6.28</param>
+            </command_interface>
+            <state_interface name="position"/>
+        </joint>
+        <joint name="left_eye_vertical_joint">
+            <command_interface name="position">
+                <param name="min">-6.28</param>
+                <param name="max">6.28</param>
+            </command_interface>
+            <state_interface name="position"/>
+        </joint>
+        <joint name="left_inferior_eyelid_joint">
+            <command_interface name="position">
+                <param name="min">-6.28</param>
+                <param name="max">6.28</param>
+            </command_interface>
+            <state_interface name="position"/>
+        </joint>
+        <joint name="left_superior_eyelid_joint">
+            <command_interface name="position">
+                <param name="min">-6.28</param>
+                <param name="max">6.28</param>
+            </command_interface>
+            <state_interface name="position"/>
+        </joint>
+        <joint name="left_vertical_eyebrow_joint">
+            <command_interface name="position">
+                <param name="min">-6.28</param>
+                <param name="max">6.28</param>
+            </command_interface>
+            <state_interface name="position"/>
+        </joint>
+        <joint name="left_rotacional_eyebrow_joint">
+            <command_interface name="position">
+                <param name="min">-6.28</param>
+                <param name="max">6.28</param>
+            </command_interface>
+            <state_interface name="position"/>
+        </joint>
+        <joint name="right_eye_horizontal_joint">
+            <command_interface name="position">
+                <param name="min">-6.28</param>
+                <param name="max">6.28</param>
+            </command_interface>
+            <state_interface name="position"/>
+        </joint>
+        <joint name="right_eye_vertical_joint">
+            <command_interface name="position">
+                <param name="min">-6.28</param>
+                <param name="max">6.28</param>
+            </command_interface>
+            <state_interface name="position"/>
+        </joint>
+        <joint name="right_inferior_eyelid_joint">
+            <command_interface name="position">
+                <param name="min">-6.28</param>
+                <param name="max">6.28</param>
+            </command_interface>
+            <state_interface name="position"/>
+        </joint>
+        <joint name="right_superior_eyelid_joint">
+            <command_interface name="position">
+                <param name="min">-6.28</param>
+                <param name="max">6.28</param>
+            </command_interface>
+            <state_interface name="position"/>
+        </joint>
+        <joint name="right_vertical_eyebrow_joint">
+            <command_interface name="position">
+                <param name="min">-6.28</param>
+                <param name="max">6.28</param>
+            </command_interface>
+            <state_interface name="position"/>
+        </joint>
+        <joint name="right_rotacional_eyebrow_joint">
+            <command_interface name="position">
+                <param name="min">-6.28</param>
+                <param name="max">6.28</param>
+            </command_interface>
+            <state_interface name="position"/>
         </joint>
     </ros2_control>

File: boris_head_description/urdf/boris_head.urdf (robot description, URDF)
Before this commit: robot boris_head, 16 links, 15 joints
Links:
- link head_link: geometry collision mesh filename=package://boris_head_description/meshes/dae/Cube.001.dae scale=0.001 0.001 0.001; visual mesh filename=package://boris_head_description/meshes/dae/Cube.001.dae scale=0.001 0.001 0.001
- link head_root: geometry collision box size=0.01 0.01 0.01
- link jaw_link: geometry collision mesh filename=package://boris_head_description/meshes/dae/Plane.012.dae scale=0.001 0.001 0.001; visual mesh filename=package://boris_head_description/meshes/dae/Plane.012.dae scale=0.001 0.001 0.001
- link left_eye_horizontal_link: geometry collision box size=0.01 0.01 0.01
- link left_eye_vertical_link: geometry collision mesh filename=package://boris_head_description/meshes/dae/Cube.002.dae scale=0.001 0.001 0.001; visual mesh filename=package://boris_head_description/meshes/dae/Cube.002.dae scale=0.001 0.001 0.001
- link left_inferior_eyelid_link: geometry collision mesh filename=package://boris_head_description/meshes/dae/Plane.015.dae scale=0.001 0.001 0.001; visual mesh filename=package://boris_head_description/meshes/dae/Plane.015.dae scale=0.001 0.001 0.001
- link left_rotacional_eyebrow_link: geometry collision mesh filename=package://boris_head_description/meshes/dae/Cylinder.004.dae scale=0.001 0.001 0.001; visual mesh filename=package://boris_head_description/meshes/dae/Cylinder.004.dae scale=0.001 0.001 0.001
- link left_superior_eyelid_link: geometry collision mesh filename=package://boris_head_description/meshes/dae/Plane.001.dae scale=0.001 0.001 0.001; visual mesh filename=package://boris_head_description/meshes/dae/Plane.001.dae scale=0.001 0.001 0.001
- link left_vertical_eyebrow_link: geometry collision box size=0.01 0.01 0.01
- link neck_link: geometry collision mesh filename=package://boris_head_description/meshes/dae/Cube.055.dae scale=0.01 0.01 0.01; visual mesh filename=package://boris_head_description/meshes/dae/Cube.055.dae scale=0.01 0.01 0.01
- link right_eye_horizontal_link: geometry collision box size=0.01 0.01 0.01
- link right_eye_vertical_link: geometry collision mesh filename=package://boris_head_description/meshes/dae/Cube.007.dae scale=0.001 0.001 0.001; visual mesh filename=package://boris_head_description/meshes/dae/Cube.007.dae scale=0.001 0.001 0.001
- link right_inferior_eyelid_link: geometry collision mesh filename=package://boris_head_description/meshes/dae/Plane.013.dae scale=0.001 0.001 0.001; visual mesh filename=package://boris_head_description/meshes/dae/Plane.013.dae scale=0.001 0.001 0.001
- link right_rotacional_eyebrow_link: geometry collision mesh filename=package://boris_head_description/meshes/dae/Cylinder.005.dae scale=0.001 0.001 0.001; visual mesh filename=package://boris_head_description/meshes/dae/Cylinder.005.dae scale=0.001 0.001 0.001
- link right_superior_eyelid_link: geometry collision mesh filename=package://boris_head_description/meshes/dae/Plane.014.dae scale=0.001 0.001 0.001; visual mesh filename=package://boris_head_description/meshes/dae/Plane.014.dae scale=0.001 0.001 0.001
- link right_vertical_eyebrow_link: geometry collision box size=0.01 0.01 0.01
