Commit message: :sparkles: first map working

File: boris_description/urdf/boris_description.xacro (robot description, xacro)
@@ -1,11 +1,12 @@
 <?xml version="1.0"?>
 <robot xmlns:xacro="http://www.ros.org/wiki/xacro" name="shark-v1">
+  <xacro:include filename="$(find shark_description)/urdf/shark.xacro" />
   <xacro:include filename="$(find sensors_description)/urdf/hokuyo.xacro" />
   <xacro:include filename="$(find sensors_description)/urdf/sick_lms1xx.xacro" />
   <xacro:include filename="$(find sensors_description)/urdf/rgb_cam.xacro" />
-  <xacro:include filename="$(find shark_description)/urdf/shark.xacro" />
   <xacro:include filename="$(find sensors_description)/urdf/realsense_camera.xacro" />
   <xacro:include filename="$(find boris_head_description)/urdf/boris_head.urdf" />
-  <xacro:include filename="$(find interbotix_xsarm_descriptions)/urdf/wx200.urdf.xacro" />
+  <!-- <xacro:include filename="$(find interbotix_xsarm_descriptions)/urdf/wx200.urdf.xacro" /> -->
+  <!-- <xacro:include filename="$(find boris_description)/ros2_control/shark_ros2_control.xacro" /> -->
   <xacro:property name="base_width" value="0.336" />
   <xacro:property name="base_len" value="0.5" />
@@ -103,9 +104,9 @@
     <origin xyz="0 0 ${dorso_height + 0.04}" rpy="0 0 0" />
   </joint>
-  <joint name="arm_to_robot" type="fixed">
+  <!-- <joint name="arm_to_robot" type="fixed">
     <origin xyz="0.1 0 ${arm_support_height/2}" rpy="0 0 0"/>
     <parent link="arm_support_link"/>
     <child link="wx200/base_link"/>
-  </joint>
+  </joint> -->
   <xacro:realsense_camera name="camera" parent="dorso_link" xyz="${dorso_len/2 + 0.05} 0 ${dorso_height + 0.053}" rpy="0 0 0"/>
   <xacro:dorso parent="base_link" depth="${dorso_len}" width="${dorso_width}" height="${dorso_height}" xyz="${-base_len/2 + (dorso_len/2)} 0 ${base_height/2}" rpy="0 0 0"/>

File: sensors_description/urdf/sick_lms1xx.xacro (robot description, xacro)
@@ -40,5 +40,5 @@
         <geometry>
           <!-- Origin of this mesh is the focal point of the LIDAR. -->
-          <mesh filename="package://lms1xx/meshes/sick-lms1xx.dae" />
+          <mesh filename="package://sensors_description/meshes/sick-lms1xx.dae" />
         </geometry>
       </visual>

File: shark_description/ros2_control/shark_ros2_control.xacro (robot description, xacro)
@@ -6,5 +6,5 @@
       <param name="wheel_radius">0.0775</param>
       <param name="max_velocity">1.0</param>
-      <param name="device">/dev/ttyUSB0</param>
+      <param name="device">/dev/ttySHARK</param>
     </hardware>
     <joint name="left_wheel_joint">

Commit message: :sparkles: added urg node and imu

File: boris_description/urdf/boris_description.xacro (robot description, xacro)
@@ -6,5 +6,5 @@
   <xacro:include filename="$(find sensors_description)/urdf/rgb_cam.xacro" />
   <xacro:include filename="$(find sensors_description)/urdf/realsense_camera.xacro" />
-  <xacro:include filename="$(find boris_head_description)/urdf/boris_head.urdf" />
+  <!-- <xacro:include filename="$(find boris_head_description)/urdf/boris_head.urdf" /> -->
   <!-- <xacro:include filename="$(find interbotix_xsarm_descriptions)/urdf/wx200.urdf.xacro" /> -->
   <!-- <xacro:include filename="$(find boris_description)/ros2_control/shark_ros2_control.xacro" /> -->
@@ -99,9 +99,9 @@
     <child link="sick_link" />
   </joint>
-  <joint name="dorso_head" type="fixed">
+  <!-- <joint name="dorso_head" type="fixed">
     <parent link="dorso_link" />
     <child link="head_root" />
     <origin xyz="0 0 ${dorso_height + 0.04}" rpy="0 0 0" />
-  </joint>
+  </joint> -->
   <!-- <joint name="arm_to_robot" type="fixed">
     <origin xyz="0.1 0 ${arm_support_height/2}" rpy="0 0 0"/>

Commit message: 💩 Version working with the hokuyo scan and sick visual but not with sick scan

File: boris_description/urdf/boris_description.xacro (robot description, xacro)
@@ -48,5 +48,5 @@
     </joint>
   </xacro:macro>
-  <xacro:sick_lms1xx />
+  <xacro:sick_lms1xx parent="base_link" xyz="${base_len/2 + 0.017 + 0.05} 0 ${0.02 + base_height/2}" rpy="0 0 0" name="sick"/>
   <xacro:macro name="dorso" params="parent depth width height xyz rpy">
     <link name="dorso_link">
@@ -94,9 +94,9 @@
     </joint>
   </xacro:macro>
-  <joint name="laser_joint" type="fixed">
+  <!-- <joint name="laser_joint" type="fixed">
     <origin xyz="${base_len/2 + 0.017 + 0.05} 0 ${0.02 + base_height/2}" rpy="0 0 0" />
     <parent link="base_link" />
     <child link="sick_link" />
-  </joint>
+  </joint> -->
   <!-- <joint name="dorso_head" type="fixed">
     <parent link="dorso_link" />

File: sensors_description/urdf/sick_lms1xx.xacro (robot description, xacro)
@@ -1,82 +1,70 @@
 <?xml version="1.0"?>
-<!--
-Copyright (c) 2013, Goncalo Cabrita, ISR University of Coimbra
-Copyright (c) 2014, 2015 Clearpath Robotics
-All rights reserved.
-Redistribution and use in source and binary forms, with or without
-modification, are permitted provided that the following conditions are met:
-    * Redistributions of source code must retain the above copyright
-      notice, this list of conditions and the following disclaimer.
-    * Redistributions in binary form must reproduce the above copyright
-      notice, this list of conditions and the following disclaimer in the
-      documentation and/or other materials provided with the distribution.
-    * Neither the name of Clearpath Robotics nor the
-      names of its contributors may be used to endorse or promote products
-      derived from this software without specific prior written permission.
-THIS SOFTWARE IS PROVIDED BY THE COPYRIGHT HOLDERS AND CONTRIBUTORS "AS IS" AND
-ANY EXPRESS OR IMPLIED WARRANTIES, INCLUDING, BUT NOT LIMITED TO, THE IMPLIED
-WARRANTIES OF MERCHANTABILITY AND FITNESS FOR A PARTICULAR PURPOSE ARE
-DISCLAIMED. IN NO EVENT SHALL THE COPYRIGHT HOLDERS BE LIABLE FOR ANY
-DIRECT, INDIRECT, INCIDENTAL, SPECIAL, EXEMPLARY, OR CONSEQUENTIAL DAMAGES
-(INCLUDING, BUT NOT LIMITED TO, PROCUREMENT OF SUBSTITUTE GOODS OR SERVICES;
-LOSS OF USE, DATA, OR PROFITS; OR BUSINESS INTERRUPTION) HOWEVER CAUSED AND
-ON ANY THEORY OF LIABILITY, WHETHER IN CONTRACT, STRICT LIABILITY, OR TORT
-(INCLUDING NEGLIGENCE OR OTHERWISE) ARISING IN ANY WAY OUT OF THE USE OF THIS
-SOFTWARE, EVEN IF ADVISED OF THE POSSIBILITY OF SUCH DAMAGE.
--->
-<robot xmlns:xacro="http://www.ros.org/wiki/xacro">
-  <xacro:macro name="sick_lms1xx" params="frame:=sick_link topic:=scan sample_size:=720 update_rate:=50
-               min_angle:=-1.570 max_angle:=1.570 min_range:=0.1 max_range:=30.0 robot_namespace:=/" >
-    <link name="${frame}">
+<robot name="sick_lms1xx"
+  xmlns:xacro="http://ros.org/wiki/xacro">
+  <xacro:macro name="sick_lms1xx" params="parent xyz rpy name frame:=sick_link topic:=scan sample_size:=720 update_rate:=50
+               min_angle:=-1.570 max_angle:=1.570 min_range:=0.1 max_range:=30.0">
+    <link name="${name}_link">
+      <!--collision>
+        <origin xyz="0 0 0" rpy="0 0 0"/>
+        <geometry>
+          <box size="0.01 0.01 0.01"/>
+        </geometry>
+      </collision-->
+      <visual>
+        <origin xyz="0 0 0" rpy="0 0 0"/>
+        <geometry>
+          <mesh filename="package://sensors_description/meshes/sick-lms1xx.dae"/>
+        </geometry>
+      </visual>
       <inertial>
         <mass value="1e-5" />
-        <origin xyz="0 0 0" />
-        <inertia ixx="1e-6" ixy="1e-20" ixz="1e-20"
-          iyy="1e-6" iyz="1e-20"
-          izz="1e-6" />
+        <origin xyz="0 0 0" rpy="0 0 0"/>
+        <inertia ixx="1e-6" ixy="0" ixz="0" iyy="1e-6" iyz="0" izz="1e-6" />
       </inertial>
-      <visual>
-        <origin xyz="0 0 0" rpy="0 0 0" />
-        <geometry>
-          <!-- Origin of this mesh is the focal point of the LIDAR. -->
-          <mesh filename="package://sensors_description/meshes/sick-lms1xx.dae" />
-        </geometry>
-      </visual>
-      <!--collision>
-        <origin xyz="0 0 -0.05" rpy="0 0 0" />
-        <geometry>
-          <box size="0.105 0.1 0.1" />
-        </geometry>
-      </collision-->
     </link>
-    <gazebo reference="${frame}">
-      <sensor type="ray" name="${frame}">
+    <joint name="${name}_joint" type="fixed">
+      <!--<axis xyz="0 0 1" />-->
+      <origin xyz="${xyz}" rpy="${rpy}"/>
+      <parent link="${parent}"/>
+      <child link="${name}_link"/>
+    </joint>
+    <!-- Hokuyo sensor for simulation -->
+    <xacro:sim_laser_range_finder/>
+  </xacro:macro>
+  <!-- ULM-30LX Hokuyo Laser Range Finder -->
+  <xacro:macro name="sim_laser_range_finder">
+    <gazebo reference="${name}_link">
+      <sensor type="ray" name="${name}">
         <pose>0 0 0 0 0 0</pose>
         <visualize>false</visualize>
-        <update_rate>${update_rate}</update_rate>
+        <update_rate>40</update_rate>
         <ray>
           <scan>
             <horizontal>
-              <samples>${sample_size}</samples>
-              <resolution>1</resolution>
-              <min_angle>${min_angle}</min_angle>
-              <max_angle>${max_angle}</max_angle>
+              <samples>683</samples>
+              <resolution>0.3515625</resolution>
+              <min_angle>-2.0943</min_angle>
+              <max_angle>2.0943</max_angle>
             </horizontal>
           </scan>
           <range>
-            <min>${min_range}</min>
-            <max>${max_range}</max>
+            <min>0.15</min>
+            <max>4.0</max>
             <resolution>0.01</resolution>
           </range>
           <noise>
             <type>gaussian</type>
+            <!-- Noise parameters based on published spec for Hokuyo laser
+               achieving "+-30mm" accuracy at range < 10m.  A mean of 0.0m and
+               stddev of 0.01m will put 99.7% of samples within 0.03m of the true
+               reading. -->
             <mean>0.0</mean>
-            <stddev>0.001</stddev>
+            <stddev>0.01</stddev>
           </noise>
         </ray>
         <plugin name="gazebo_ros_laser" filename="libgazebo_ros_laser.so">
-          <topicName>${topic}</topicName>
-          <frameName>${frame}</frameName>
-          <robotNamespace>${robot_namespace}</robotNamespace>
+          <topicName>scan</topicName>
+          <frameName>${name}_link</frameName>
+          <robotNamespace>/</robotNamespace>
         </plugin>
       </sensor>

File: shark_description/ros2_control/shark_ros2_control.xacro (robot description, xacro)
@@ -6,5 +6,5 @@
       <param name="wheel_radius">0.0775</param>
       <param name="max_velocity">1.0</param>
-      <param name="device">/dev/ttySHARK</param>
+      <param name="device">/dev/ttyUSB0</param>
     </hardware>
     <joint name="left_wheel_joint">

Commit message: :poop: workng version with hokuyo, without sick visuals

File: boris_description/urdf/boris_description.xacro (robot description, xacro)
@@ -3,5 +3,5 @@
   <xacro:include filename="$(find shark_description)/urdf/shark.xacro" />
   <xacro:include filename="$(find sensors_description)/urdf/hokuyo.xacro" />
-  <xacro:include filename="$(find sensors_description)/urdf/sick_lms1xx.xacro" />
+  <xacro:include filename="/home/stihl/fbot_ws/src/sick_scan_xd/urdf/sick_lms1xx.urdf.xacro" />
   <xacro:include filename="$(find sensors_description)/urdf/rgb_cam.xacro" />
   <xacro:include filename="$(find sensors_description)/urdf/realsense_camera.xacro" />
@@ -48,5 +48,5 @@
     </joint>
   </xacro:macro>
-  <xacro:sick_lms1xx />
+  <xacro:sick_lms_1xx name="sick" ros_topic="/scan" />
   <xacro:macro name="dorso" params="parent depth width height xyz rpy">
     <link name="dorso_link">
@@ -97,5 +97,5 @@
     <origin xyz="${base_len/2 + 0.017 + 0.05} 0 ${0.02 + base_height/2}" rpy="0 0 0" />
     <parent link="base_link" />
-    <child link="sick_link" />
+    <child link="sick_mount_link" />
   </joint>
   <!-- <joint name="dorso_head" type="fixed">

File: shark_description/ros2_control/shark_ros2_control.xacro (robot description, xacro)
@@ -6,5 +6,5 @@
       <param name="wheel_radius">0.0775</param>
       <param name="max_velocity">1.0</param>
-      <param name="device">/dev/ttySHARK</param>
+      <param name="device">/dev/ttyUSB1</param>
     </hardware>
     <joint name="left_wheel_joint">

Commit message: Add caster wheel for gazebo simulation

File: boris_description/urdf/boris_description.xacro (robot description, xacro)
@@ -2,10 +2,7 @@
 <robot xmlns:xacro="http://www.ros.org/wiki/xacro" name="shark-v1">
   <xacro:include filename="$(find shark_description)/urdf/shark.xacro" />
-  <xacro:include filename="$(find sensors_description)/urdf/hokuyo.xacro" />
-  <xacro:include filename="$(find sensors_description)/urdf/sick_lms1xx.urdf.xacro" />
-  <xacro:include filename="$(find sensors_description)/urdf/rgb_cam.xacro" />
-  <xacro:include filename="$(find sensors_description)/urdf/realsense_camera.xacro" />
-  <!-- <xacro:include filename="$(find boris_head_description)/urdf/boris_head.urdf" /> -->
-  <!-- <xacro:include filename="$(find interbotix_xsarm_descriptions)/urdf/wx200.urdf.xacro" /> -->
+  <xacro:include filename="$(find sensors_description)/urdf/realsense_camera.urdf.xacro" />
+  <xacro:include filename="$(find boris_head_description)/urdf/boris_head.urdf" />
+  <xacro:include filename="$(find boris_head_description)/urdf/control.urdf.xacro" />
   <!-- <xacro:include filename="$(find boris_description)/ros2_control/shark_ros2_control.xacro" /> -->
   <xacro:property name="base_width" value="0.336" />
@@ -48,5 +45,9 @@
     </joint>
   </xacro:macro>
+<<<<<<< HEAD:boris_description/urdf/boris_description.xacro
   <xacro:sick_lms_1xx name="sick" ros_topic="/scan" />
+=======
+  <xacro:sick_lms1xx robot_namespace="/lms1xx" />
+>>>>>>> 46ae7d8 (Add caster wheel for gazebo simulation):boris_description/urdf/boris.xacro
   <xacro:macro name="dorso" params="parent depth width height xyz rpy">
     <link name="dorso_link">
@@ -70,7 +71,6 @@
         <child link="dorso_link"/>
         <origin xyz="${xyz}" rpy="${rpy}"/>
-    </joint>0
+    </joint>
   </xacro:macro>
-    <!--32,5-->
   <xacro:macro name="arm_support" params="parent width height depth xyz rpy">
     <link name="arm_support_link">
@@ -104,4 +104,5 @@
     <origin xyz="0 0 ${dorso_height + 0.04}" rpy="0 0 0" />
   </joint> -->
+<<<<<<< HEAD:boris_description/urdf/boris_description.xacro
   <!-- <joint name="arm_to_robot" type="fixed">
     <origin xyz="0.1 0 ${arm_support_height/2}" rpy="0 0 0"/>
@@ -118,8 +119,16 @@
     </xacro:macro>
   <xacro:realsense_camera name="camera" parent="dorso_link" xyz="${dorso_len/2 + 0.05} 0 ${dorso_height + 0.053}" rpy="0 0 0"/>
+=======
+  <xacro:realsense_camera name="camera" parent="dorso_link">
+    <origin xyz="${dorso_len/2 + 0.05} 0 ${dorso_height + 0.053}" rpy="0 0 ${3.14/8}" />
+  </xacro:realsense_camera>
+  <xacro:realsense_gazebo />
+  <xacro:add_optical_frame name="camera_link" />
+>>>>>>> 46ae7d8 (Add caster wheel for gazebo simulation):boris_description/urdf/boris.xacro
   <xacro:dorso parent="base_link" depth="${dorso_len}" width="${dorso_width}" height="${dorso_height}" xyz="${-base_len/2 + (dorso_len/2)} 0 ${base_height/2}" rpy="0 0 0"/>
   <xacro:arm_support parent="dorso_link" width="${arm_support_width}" height="${arm_support_height}" depth="${arm_support_len}" xyz="${dorso_len/2 + arm_support_len/2} 0 ${arm_z_position}" rpy="0 0 0"/>
   <xacro:sensor_hokuyo parent="base_link" xyz="${base_len/2 + 0.017 + 0.024} 0 ${0.02 - base_height/2}" rpy="3.14 0 0" name="ground"/>
   <xacro:sensor_hokuyo parent="base_link" xyz="${-base_len/2 - 0.017 - 0.024} 0 ${0.02 - base_height/2}" rpy="3.14 0 3.14" name="back"/>
+<<<<<<< HEAD:boris_description/urdf/boris_description.xacro
   <!-- <xacro:imu parent="base_link" xyz="-0.01 0 ${0.02 - base_height/2}" rpy="-0.014161 -0.0203861 0" /> -->
   <!-- <xacro:boris_arm parent="arm_support_link" xyz="0.1 0 ${arm_support_height/2}" rpy="0 0 0"/> -->
@@ -128,2 +137,12 @@
   <xacro:shark_base/>  <!-- isso aq n existe mais, a gente reverteu as mudanças do luis que transformavam aquilo tudo em um macro q n ta aparecendo mais -->
 </robot>
+=======
+  <xacro:imu parent="base_link" xyz="-0.01 0 ${0.02 - base_height/2}" rpy="-0.014161 -0.0203861 0" />
+  <gazebo reference="dorso_link">
+    <material>Gazebo/DarkGray</material>
+  </gazebo>
+  <gazebo reference="arm_support_link">
+    <material>Gazebo/DarkGray</material>
+  </gazebo>
+</robot>
+>>>>>>> 46ae7d8 (Add caster wheel for gazebo simulation):boris_description/urdf/boris.xacro

File: sensors_description/urdf/realsense_camera.xacro (robot description, xacro)
@@ -2,6 +2,81 @@
 <robot name="realsense_rgbd" xmlns:xacro="http://www.ros.org/wiki/xacro">
   <xacro:property name="M_PI" value="3.1415926535897931"/>
+  <xacro:macro name="add_optical_frame" params="name">
+		<joint name="${name}_optical_joint" type="fixed">
+			<origin xyz="0 0 0" rpy="0.0 0.0 0.0" />
+			<parent link="${name}" />
+			<child link="${name}_optical_frame"/>
+		</joint>
+		<link name="${name}_optical_frame" />
+	</xacro:macro>
+  <xacro:macro name="realsense_gazebo">
+		<gazebo reference="camera_link_optical_frame">
+			<sensor type="camera" name="realsense">
+				<always_on>true</always_on>
+				<visualize>true</visualize>
+				<update_rate>15</update_rate>
+				<gz_frame_id>camera_link_optical_frame</gz_frame_id>
+				<camera>
+					<optical_frame_id>camera_link_optical_frame</optical_frame_id>
+					<horizontal_fov>1.047</horizontal_fov>
+					<image>
+						<width>640</width>
+						<height>480</height>
+					</image>
+					<depth_camera>
+						<clip>
+							<near>0.1</near>
+							<far>10.0</far>
+						</clip>
+					</depth_camera>
+					<noise>
+						<type>gaussian</type>
+						<mean>0.0</mean>
+						<stddev>0.01</stddev>
+					</noise>
+				</camera>
+                <plugin name="realsense_camera_plugin" filename="libgazebo_ros_camera.so">
+                    <ros>
+                    <remapping>image_raw:=/realsense/image_color/raw</remapping>
+                    <remapping>camera_info:=/realsense/image_color/camera_info</remapping>
+                    <frame_name>camera_link_optical_frame</frame_name>
+                    </ros>
+                </plugin>
+			</sensor>
+            <sensor type="depth" name="realsense_depth">
+				<always_on>true</always_on>
+				<visualize>true</visualize>
+				<update_rate>15</update_rate>
+				<gz_frame_id>camera_link_optical_frame</gz_frame_id>
+				<camera>
+					<optical_frame_id>camera_link_optical_frame</optical_frame_id>
+					<horizontal_fov>1.047</horizontal_fov>
+					<image>
+						<width>640</width>
+						<height>480</height>
+					</image>
+					<depth_camera>
+						<clip>
+							<near>0.1</near>
+							<far>10.0</far>
+						</clip>
+					</depth_camera>
+					<noise>
+						<type>gaussian</type>
+						<mean>0.0</mean>
+						<stddev>0.01</stddev>
+					</noise>
+				</camera>
+                <plugin name="realsense_camera_plugin" filename="libgazebo_ros_camera.so">
+                    <ros>
+                    <remapping>image_raw:=/realsense/image_depth/raw</remapping>
+                    <remapping>camera_info:=/realsense/image_depth/camera_info</remapping>
+                    <frame_name>camera_link_optical_frame</frame_name>
+                    </ros>
+                </plugin>
+			</sensor>
+		</gazebo>
+	</xacro:macro>
   <xacro:macro name="realsense_camera" params="name parent xyz rpy">
-      <!-- @TODO: GABIARRA PRA GIRAR A CAMERA -->
       <link name="head_pan_link_static">
           <inertial>
@@ -131,7 +206,19 @@
           <axis xyz="0 0 0"/>
       </joint>
-      <!-- <xacro:sensor_d435 parent="head_tilt_link" use_nominal_extrinsics="false" add_plug="false" use_mesh="true">
-          <origin xyz="0.06705 0 -0.00425" rpy="0 0 0"/>
-      </xacro:sensor_d435> -->
+      <ros2_control name="head_hardware_interface" type="system">
+    <hardware>
+      <plugin>gazebo_ros2_control/GazeboSystem</plugin>
+    </hardware>
+    <joint name="head_pan_joint">
+      <command_interface name="position">
+      </command_interface>
+      <state_interface name="position"/>
+    </joint>
+    <joint name="head_tilt_joint">
+      <command_interface name="position">
+      </command_interface>
+      <state_interface name="position"/>
+    </joint>
+  </ros2_control>
   </xacro:macro>
 </robot>

File: shark_description/urdf/shark_description.xacro (robot description, xacro)
@@ -10,4 +10,6 @@
   <xacro:property name="wheel_joint_offset" value="0.0" />
   <xacro:property name="caster_height" value="0.07" />
+  <xacro:property name="caster_wheel_joint_offset" value="0.0" />
+  <xacro:property name="caster_wheel_radius" value="0.02" />
   <xacro:macro name="box_inertia" params="m w h d">
     <inertial>
@@ -39,5 +41,5 @@
       <xacro:cylinder_inertia m="10" r="${wheel_radius}" h="0.05"/>
     </link>
-    <joint name="${prefix}_wheel" type="continuous">
+    <joint name="${prefix}_wheel_joint" type="continuous">
       <axis xyz="0 1 0" rpy="0 0 0" />
       <parent link="base_link"/>
@@ -52,27 +54,25 @@
     </inertial>
   </xacro:macro>
-  <xacro:macro name="shark_base">
-    <link name="base_footprint"/>
-    <link name="base_link">
-      <xacro:box_inertia m="1" w="${base_len}" h="${base_width}" d="0.01" />
-      <visual>
-        <material name="lightgray" />
-        <geometry>
-          <box size="${base_len} ${base_width} ${base_height}" />
-        </geometry>
-      </visual>
-      <collision>
-        <geometry>
-          <box size="${base_len} ${base_width} ${base_height}" />
-        </geometry>
-      </collision>
-    </link>
-    <joint name="base_link_joint" type="fixed">
-      <origin xyz="0 0 ${base_height/2 + caster_height}" rpy="0 0 0" />
-      <parent link="base_footprint" />
-      <child link="base_link" />
-    </joint>
-    <xacro:wheel prefix="left" reflect="1" />
-    <xacro:wheel prefix="right" reflect="-1" />
-  </xacro:macro>
+   <link name="caster_wheel">
+     <visual>
+       <material name="darkgray"/>
+      <origin xyz="0 0 0" rpy="0 0 0"/>
+      <geometry>
+        <sphere radius="${caster_wheel_radius}"/>
+      </geometry>
+    </visual>
+    <collision>
+      <origin xyz="0 0 0" rpy="0 0 0"/>
+      <geometry>
+        <sphere radius="${caster_wheel_radius}"/>
+      </geometry>
+    </collision>
+    <xacro:sphere_inertia m="5" r="${caster_wheel_radius}"/>
+  </link>
+  <joint name="caster_wheel_joint" type="continuous">
+    <axis xyz="0 1 0" rpy="0 0 0" />
+    <parent link="base_link"/>
+    <child link="caster_wheel"/>
+    <origin xyz="${(base_len/2) - caster_wheel_joint_offset} 0 ${(caster_wheel_radius - caster_height) - base_height/2}" rpy="0 0 0"/>
+  </joint>
 </robot>
