Commit message: changes to xacros

File: boris_description/urdf/boris_description.xacro (robot description, xacro)
@@ -1,4 +1,10 @@
 <?xml version="1.0"?>
 <robot xmlns:xacro="http://www.ros.org/wiki/xacro" name="shark-v1">
+  <xacro:include filename="$(find sensors_description)/urdf/hokuyo.xacro" />
+  <xacro:include filename="$(find sensors_description)/urdf/sick_lms1xx.xacro" />
+  <xacro:include filename="$(find sensors_description)/urdf/rgb_cam.xacro" />
+  <xacro:include filename="$(find sensors_description)/urdf/camera_turret.xacro" />
+  <xacro:include filename="$(find hector_models)/urdf/orbbec_astra2.xacro" />
+  <xacro:include filename="$(find hector_models)/gazebo/orbbec_astra2.gazebo.xacro" />
   <xacro:include filename="$(find shark_description)/urdf/shark.xacro" />
   <xacro:include filename="$(find sensors_description)/urdf/realsense_camera.urdf.xacro" />
@@ -105,4 +111,5 @@
   </joint> -->
 <<<<<<< HEAD:boris_description/urdf/boris_description.xacro
+<<<<<<< HEAD:boris_description/urdf/boris_description.xacro
   <!-- <joint name="arm_to_robot" type="fixed">
     <origin xyz="0.1 0 ${arm_support_height/2}" rpy="0 0 0"/>
@@ -126,4 +133,14 @@
   <xacro:add_optical_frame name="camera_link" />
 >>>>>>> 46ae7d8 (Add caster wheel for gazebo simulation):boris_description/urdf/boris.xacro
+=======
+  <xacro:camera_turret parent="dorso_link" name="camera_turret">
+    <origin xyz="${dorso_len/2 + 0.05} 0 ${dorso_height + 0.053}" rpy="0 0 ${3.14/8}" />
+  </xacro:camera_turret>
+  <xacro:orbbec_astra2 name="top_camera">
+    <parent link="camera_turret_tilt_link"/>
+    <origin rpy="0 0 0" xyz="0.06705 0 -0.00425"/>
+  </xacro:orbbec_astra2>
+  <xacro:orbbec_astra2_gazebo name="top_camera" semantic_segmentation="false"/>
+>>>>>>> d617c95 (changes to xacros):boris_description/urdf/boris.xacro
   <xacro:dorso parent="base_link" depth="${dorso_len}" width="${dorso_width}" height="${dorso_height}" xyz="${-base_len/2 + (dorso_len/2)} 0 ${base_height/2}" rpy="0 0 0"/>
   <xacro:arm_support parent="dorso_link" width="${arm_support_width}" height="${arm_support_height}" depth="${arm_support_len}" xyz="${dorso_len/2 + arm_support_len/2} 0 ${arm_z_position}" rpy="0 0 0"/>

File: shark_description/urdf/shark_description.xacro (robot description, xacro)
@@ -18,4 +18,25 @@
     </inertial>
   </xacro:macro>
+  <link name="base_footprint">
+  </link>
+  <link name="base_link">
+    <xacro:box_inertia m="1" w="${base_len}" h="${base_width}" d="0.01"/>
+    <visual>
+      <material name="lightgray"/>
+      <geometry>
+        <box size="${base_len} ${base_width} ${base_height}"/>
+      </geometry>
+    </visual>
+    <collision>
+      <geometry>
+        <box size="${base_len} ${base_width} ${base_height}"/>
+      </geometry>
+    </collision>
+  </link>
+  <joint name="base_link_joint" type="fixed">
+    <origin xyz="0 0 ${base_height/2 + caster_height}" rpy="0 0 0" />
+    <parent link="base_footprint"/>
+    <child link="base_link" />
+  </joint>
   <xacro:macro name="cylinder_inertia" params="m r h">
     <inertial>

Commit message: :construction: Adding imu again, adding use_rviz flag to sick launch, and adding hokuyo usb rules

File: boris_description/urdf/boris_description.xacro (robot description, xacro)
@@ -109,4 +109,12 @@
     <child link="wx200/base_link"/>
   </joint> -->
+    <xacro:macro name="imu" params="parent xyz rpy">
+    <link name="imu_link"/>
+    <joint name="imu_joint" type="fixed">
+      <parent link="${parent}"/>
+      <child link="imu_link"/>
+      <origin xyz="${xyz}" rpy="${rpy}"/>
+    </joint>
+    </xacro:macro>
   <xacro:realsense_camera name="camera" parent="dorso_link" xyz="${dorso_len/2 + 0.05} 0 ${dorso_height + 0.053}" rpy="0 0 0"/>
   <xacro:dorso parent="base_link" depth="${dorso_len}" width="${dorso_width}" height="${dorso_height}" xyz="${-base_len/2 + (dorso_len/2)} 0 ${base_height/2}" rpy="0 0 0"/>
@@ -114,7 +122,8 @@
   <xacro:sensor_hokuyo parent="base_link" xyz="${base_len/2 + 0.017 + 0.024} 0 ${0.02 - base_height/2}" rpy="3.14 0 0" name="ground"/>
   <xacro:sensor_hokuyo parent="base_link" xyz="${-base_len/2 - 0.017 - 0.024} 0 ${0.02 - base_height/2}" rpy="3.14 0 3.14" name="back"/>
-  <xacro:imu parent="base_link" xyz="-0.01 0 ${0.02 - base_height/2}" rpy="-0.014161 -0.0203861 0" />
+  <!-- <xacro:imu parent="base_link" xyz="-0.01 0 ${0.02 - base_height/2}" rpy="-0.014161 -0.0203861 0" /> -->
   <!-- <xacro:boris_arm parent="arm_support_link" xyz="0.1 0 ${arm_support_height/2}" rpy="0 0 0"/> -->
   <!-- <xacro:rgb_cam parent="wx200/gripper_bar_link" name="webcam" xyz="-0.078 0.0 0.05" rpy="0 0 0"/> -->
+  <xacro:imu parent="base_link" xyz="${base_len/2 + 0.0625} 0 ${0.02 - base_height/2}" rpy="0 0 0"/>
   <xacro:shark_base/>  <!-- isso aq n existe mais, a gente reverteu as mudanças do luis que transformavam aquilo tudo em um macro q n ta aparecendo mais -->
 </robot>

Commit message: Changes to make it possible to simulate Boris on Ignition.

File: boris_description/urdf/boris_description.xacro (robot description, xacro)
@@ -51,9 +51,5 @@
     </joint>
   </xacro:macro>
-<<<<<<< HEAD:boris_description/urdf/boris_description.xacro
-  <xacro:sick_lms_1xx name="sick" ros_topic="/scan" />
-=======
   <xacro:sick_lms1xx robot_namespace="/lms1xx" />
->>>>>>> 46ae7d8 (Add caster wheel for gazebo simulation):boris_description/urdf/boris.xacro
   <xacro:macro name="dorso" params="parent depth width height xyz rpy">
     <link name="dorso_link">
@@ -139,8 +135,12 @@
   <xacro:orbbec_astra2 name="top_camera">
     <parent link="camera_turret_tilt_link"/>
-    <origin rpy="0 0 0" xyz="0.06705 0 -0.00425"/>
+    <origin rpy="0 0 -${M_PI/6}" xyz="0.06705 0 -0.00425"/>
   </xacro:orbbec_astra2>
+<<<<<<< HEAD:boris_description/urdf/boris_description.xacro
   <xacro:orbbec_astra2_gazebo name="top_camera" semantic_segmentation="false"/>
 >>>>>>> d617c95 (changes to xacros):boris_description/urdf/boris.xacro
+=======
+  <xacro:orbbec_astra2_gazebo name="top_camera"/>
+>>>>>>> f3a188e (Changes to make it possible to simulate Boris on Ignition.):boris_description/urdf/boris.xacro
   <xacro:dorso parent="base_link" depth="${dorso_len}" width="${dorso_width}" height="${dorso_height}" xyz="${-base_len/2 + (dorso_len/2)} 0 ${base_height/2}" rpy="0 0 0"/>
   <xacro:arm_support parent="dorso_link" width="${arm_support_width}" height="${arm_support_height}" depth="${arm_support_len}" xyz="${dorso_len/2 + arm_support_len/2} 0 ${arm_z_position}" rpy="0 0 0"/>

Commit message: :construction: adding arm on URDF

File: boris_description/urdf/boris_description.xacro (robot description, xacro)
@@ -7,5 +7,5 @@
   <xacro:include filename="$(find sensors_description)/urdf/realsense_camera.xacro" />
   <!-- <xacro:include filename="$(find boris_head_description)/urdf/boris_head.urdf" /> -->
-  <!-- <xacro:include filename="$(find interbotix_xsarm_descriptions)/urdf/wx200.urdf.xacro" /> -->
+  <xacro:include filename="$(find interbotix_xsarm_descriptions)/urdf/wx200.urdf.xacro" />
   <!-- <xacro:include filename="$(find boris_description)/ros2_control/shark_ros2_control.xacro" /> -->
   <xacro:property name="base_width" value="0.336" />
@@ -104,9 +104,9 @@
     <origin xyz="0 0 ${dorso_height + 0.04}" rpy="0 0 0" />
   </joint> -->
-  <!-- <joint name="arm_to_robot" type="fixed">
+  <joint name="arm_to_robot" type="fixed">
     <origin xyz="0.1 0 ${arm_support_height/2}" rpy="0 0 0"/>
     <parent link="arm_support_link"/>
     <child link="wx200/base_link"/>
-  </joint> -->
+  </joint>
     <xacro:macro name="imu" params="parent xyz rpy">
     <link name="imu_link"/>
