Commit message: turned shark into macro

File: shark_description/urdf/shark_description.xacro (robot description, xacro)
@@ -12,41 +12,14 @@
   <xacro:macro name="box_inertia" params="m w h d">
     <inertial>
-      <mass value="${m}"/>
-      <inertia ixx="${m / 12.0 * (d*d + h*h)}" ixy="0.0" ixz="0.0" iyy="${m / 12.0 * (w*w + h*h)}" iyz="0.0" izz="${m / 12.0 * (w*w + d*d)}"/>
+      <mass value="${m}" />
+      <inertia ixx="${m / 12.0 * (d*d + h*h)}" ixy="0.0" ixz="0.0" iyy="${m / 12.0 * (w*w + h*h)}"
+        iyz="0.0" izz="${m / 12.0 * (w*w + d*d)}" />
     </inertial>
   </xacro:macro>
-  <link name="base_footprint">
-    <xacro:box_inertia m="8" w="0.001" h="0.001" d="0.001"/>
-    <visual>
-      <origin xyz="0 0 0" rpy="0 0 0" />
-      <material name="white"/>
-        <geometry>
-            <box size="0.001 0.001 0.001" />
-        </geometry>
-    </visual>
-  </link>
-  <link name="base_link">
-    <xacro:box_inertia m="1" w="${base_len}" h="${base_width}" d="0.01"/>
-    <visual>
-      <material name="lightgray"/>
-      <geometry>
-        <box size="${base_len} ${base_width} ${base_height}"/>
-      </geometry>
-    </visual>
-    <collision>
-      <geometry>
-        <box size="${base_len} ${base_width} ${base_height}"/>
-      </geometry>
-    </collision>
-  </link>
-  <joint name="base_link_joint" type="fixed">
-    <origin xyz="0 0 ${base_height/2 + caster_height}" rpy="0 0 0" />
-    <parent link="base_footprint"/>
-    <child link="base_link" />
-  </joint>
   <xacro:macro name="cylinder_inertia" params="m r h">
     <inertial>
-      <mass value="${m}"/>
-      <inertia ixx="${m*(3*r*r+h*h)/12}" ixy = "0" ixz = "0" iyy="${m*(3*r*r+h*h)/12}" iyz = "0" izz="${m*r*r/2}"/>
+      <mass value="${m}" />
+      <inertia ixx="${m*(3*r*r+h*h)/12}" ixy="0" ixz="0" iyy="${m*(3*r*r+h*h)/12}" iyz="0"
+        izz="${m*r*r/2}" />
     </inertial>
   </xacro:macro>
@@ -54,54 +27,67 @@
     <link name="${prefix}_wheel">
       <visual>
-	      <material name="darkgray"/>
-        <origin xyz="0 0 0" rpy="${pi/2} 0 0"/>
+        <material name="darkgray" />
+        <origin xyz="0 0 0" rpy="${pi/2} 0 0" />
         <geometry>
-          <cylinder radius="${wheel_radius}" length="${wheel_width}"/>
+          <cylinder radius="${wheel_radius}" length="${wheel_width}" />
         </geometry>
       </visual>
       <collision>
-        <origin xyz="0 0 0" rpy="${pi/2} 0 0"/>
+        <origin xyz="0 0 0" rpy="${pi/2} 0 0" />
         <geometry>
-          <cylinder radius="${wheel_radius}" length="0.05"/>
+          <cylinder radius="${wheel_radius}" length="0.05" />
         </geometry>
       </collision>
-      <xacro:cylinder_inertia m="10" r="${wheel_radius}" h="0.05"/>
+      <xacro:cylinder_inertia m="10" r="${wheel_radius}" h="0.05" />
     </link>
     <joint name="${prefix}_wheel" type="continuous">
       <axis xyz="0 1 0" rpy="0 0 0" />
-      <parent link="base_link"/>
-      <child link="${prefix}_wheel"/>
-      <origin xyz="${wheel_joint_offset} ${((base_width/2)+base_wheel_gap)*reflect} ${(wheel_radius - caster_height) - base_height/2}" rpy="0 0 0"/>
+      <parent link="base_link" />
+      <child link="${prefix}_wheel" />
+      <origin
+        xyz="${wheel_joint_offset} ${((base_width/2)+base_wheel_gap)*reflect} ${(wheel_radius - caster_height) - base_height/2}"
+        rpy="0 0 0" />
     </joint>
   </xacro:macro>
-  <xacro:wheel prefix="left" reflect="1"/>
-  <xacro:wheel prefix="right" reflect="-1"/>
   <xacro:macro name="sphere_inertia" params="m r">
     <inertial>
-      <mass value="${m}"/>
-      <inertia ixx="${2.0*m*(r*r)/5.0}" ixy="0.0" ixz="0.0" iyy="${2.0*m*(r*r)/5.0}" iyz="0.0" izz="${2.0*m*(r*r)/5.0}"/>
+      <mass value="${m}" />
+      <inertia ixx="${2.0*m*(r*r)/5.0}" ixy="0.0" ixz="0.0" iyy="${2.0*m*(r*r)/5.0}" iyz="0.0"
+        izz="${2.0*m*(r*r)/5.0}" />
     </inertial>
   </xacro:macro>
-   <!-- <link name="caster_wheel">
-     <visual>
-       <material name="darkgray"/>
-      <origin xyz="0 0 0" rpy="0 0 0"/>
-      <geometry>
-        <sphere radius="${caster_wheel_radius}"/>
-      </geometry>
-    </visual>
-    <collision>
-      <origin xyz="0 0 0" rpy="0 0 0"/>
-      <geometry>
-        <sphere radius="${caster_wheel_radius}"/>
-      </geometry>
-    </collision>
-    <xacro:sphere_inertia m="5" r="${caster_wheel_radius}"/>
-  </link>
-  <joint name="caster_wheel_joint" type="continuous">
-    <axis xyz="0 1 0" rpy="0 0 0" />
-    <parent link="base_link"/>
-    <child link="caster_wheel"/>
-    <origin xyz="${caster_wheel_joint_offset} 0 -${0.06+caster_wheel_radius}" rpy="0 0 0"/>
-  </joint> -->
+  <xacro:macro name="shark_base">
+    <link name="base_footprint">
+      <xacro:box_inertia m="8" w="0.001" h="0.001" d="0.001" />
+      <visual>
+        <origin xyz="0 0 0" rpy="0 0 0" />
+        <material name="white" />
+        <geometry>
+          <box size="0.001 0.001 0.001" />
+        </geometry>
+      </visual>
+    </link>
+    <link name="base_link">
+      <xacro:box_inertia m="1" w="${base_len}" h="${base_width}" d="0.01" />
+      <visual>
+        <material name="lightgray" />
+        <geometry>
+          <box size="${base_len} ${base_width} ${base_height}" />
+        </geometry>
+      </visual>
+      <collision>
+        <geometry>
+          <box size="${base_len} ${base_width} ${base_height}" />
+        </geometry>
+      </collision>
+    </link>
+    <joint name="base_link_joint" type="fixed">
+      <origin xyz="0 0 ${base_height/2 + caster_height}" rpy="0 0 0" />
+      <parent link="base_footprint" />
+      <child link="base_link" />
+    </joint>
+    <xacro:wheel prefix="left" reflect="1" />
+    <xacro:wheel prefix="right" reflect="-1" />
+  </xacro:macro>
+  <xacro:shark_base/>
 </robot>

Commit message: base_footprint link restored

File: shark_description/urdf/shark_description.xacro (robot description, xacro)
@@ -12,14 +12,41 @@
   <xacro:macro name="box_inertia" params="m w h d">
     <inertial>
-      <mass value="${m}" />
-      <inertia ixx="${m / 12.0 * (d*d + h*h)}" ixy="0.0" ixz="0.0" iyy="${m / 12.0 * (w*w + h*h)}"
-        iyz="0.0" izz="${m / 12.0 * (w*w + d*d)}" />
+      <mass value="${m}"/>
+      <inertia ixx="${m / 12.0 * (d*d + h*h)}" ixy="0.0" ixz="0.0" iyy="${m / 12.0 * (w*w + h*h)}" iyz="0.0" izz="${m / 12.0 * (w*w + d*d)}"/>
     </inertial>
   </xacro:macro>
+  <link name="base_footprint">
+    <xacro:box_inertia m="8" w="0.001" h="0.001" d="0.001"/>
+    <visual>
+      <origin xyz="0 0 0" rpy="0 0 0" />
+      <material name="white"/>
+        <geometry>
+            <box size="0.001 0.001 0.001" />
+        </geometry>
+    </visual>
+  </link>
+  <link name="base_link">
+    <xacro:box_inertia m="1" w="${base_len}" h="${base_width}" d="0.01"/>
+    <visual>
+      <material name="lightgray"/>
+      <geometry>
+        <box size="${base_len} ${base_width} ${base_height}"/>
+      </geometry>
+    </visual>
+    <collision>
+      <geometry>
+        <box size="${base_len} ${base_width} ${base_height}"/>
+      </geometry>
+    </collision>
+  </link>
+  <joint name="base_link_joint" type="fixed">
+    <origin xyz="0 0 ${base_height/2 + caster_height}" rpy="0 0 0" />
+    <parent link="base_footprint"/>
+    <child link="base_link" />
+  </joint>
   <xacro:macro name="cylinder_inertia" params="m r h">
     <inertial>
-      <mass value="${m}" />
-      <inertia ixx="${m*(3*r*r+h*h)/12}" ixy="0" ixz="0" iyy="${m*(3*r*r+h*h)/12}" iyz="0"
-        izz="${m*r*r/2}" />
+      <mass value="${m}"/>
+      <inertia ixx="${m*(3*r*r+h*h)/12}" ixy = "0" ixz = "0" iyy="${m*(3*r*r+h*h)/12}" iyz = "0" izz="${m*r*r/2}"/>
     </inertial>
   </xacro:macro>
@@ -27,67 +54,54 @@
     <link name="${prefix}_wheel">
       <visual>
-        <material name="darkgray" />
-        <origin xyz="0 0 0" rpy="${pi/2} 0 0" />
+	      <material name="darkgray"/>
+        <origin xyz="0 0 0" rpy="${pi/2} 0 0"/>
         <geometry>
-          <cylinder radius="${wheel_radius}" length="${wheel_width}" />
+          <cylinder radius="${wheel_radius}" length="${wheel_width}"/>
         </geometry>
       </visual>
       <collision>
-        <origin xyz="0 0 0" rpy="${pi/2} 0 0" />
+        <origin xyz="0 0 0" rpy="${pi/2} 0 0"/>
         <geometry>
-          <cylinder radius="${wheel_radius}" length="0.05" />
+          <cylinder radius="${wheel_radius}" length="0.05"/>
         </geometry>
       </collision>
-      <xacro:cylinder_inertia m="10" r="${wheel_radius}" h="0.05" />
+      <xacro:cylinder_inertia m="10" r="${wheel_radius}" h="0.05"/>
     </link>
     <joint name="${prefix}_wheel" type="continuous">
       <axis xyz="0 1 0" rpy="0 0 0" />
-      <parent link="base_link" />
-      <child link="${prefix}_wheel" />
-      <origin
-        xyz="${wheel_joint_offset} ${((base_width/2)+base_wheel_gap)*reflect} ${(wheel_radius - caster_height) - base_height/2}"
-        rpy="0 0 0" />
+      <parent link="base_link"/>
+      <child link="${prefix}_wheel"/>
+      <origin xyz="${wheel_joint_offset} ${((base_width/2)+base_wheel_gap)*reflect} ${(wheel_radius - caster_height) - base_height/2}" rpy="0 0 0"/>
     </joint>
   </xacro:macro>
+  <xacro:wheel prefix="left" reflect="1"/>
+  <xacro:wheel prefix="right" reflect="-1"/>
   <xacro:macro name="sphere_inertia" params="m r">
     <inertial>
-      <mass value="${m}" />
-      <inertia ixx="${2.0*m*(r*r)/5.0}" ixy="0.0" ixz="0.0" iyy="${2.0*m*(r*r)/5.0}" iyz="0.0"
-        izz="${2.0*m*(r*r)/5.0}" />
+      <mass value="${m}"/>
+      <inertia ixx="${2.0*m*(r*r)/5.0}" ixy="0.0" ixz="0.0" iyy="${2.0*m*(r*r)/5.0}" iyz="0.0" izz="${2.0*m*(r*r)/5.0}"/>
     </inertial>
   </xacro:macro>
-  <xacro:macro name="shark_base">
-    <link name="base_footprint">
-      <xacro:box_inertia m="8" w="0.001" h="0.001" d="0.001" />
-      <visual>
-        <origin xyz="0 0 0" rpy="0 0 0" />
-        <material name="white" />
-        <geometry>
-          <box size="0.001 0.001 0.001" />
-        </geometry>
-      </visual>
-    </link>
-    <link name="base_link">
-      <xacro:box_inertia m="1" w="${base_len}" h="${base_width}" d="0.01" />
-      <visual>
-        <material name="lightgray" />
-        <geometry>
-          <box size="${base_len} ${base_width} ${base_height}" />
-        </geometry>
-      </visual>
-      <collision>
-        <geometry>
-          <box size="${base_len} ${base_width} ${base_height}" />
-        </geometry>
-      </collision>
-    </link>
-    <joint name="base_link_joint" type="fixed">
-      <origin xyz="0 0 ${base_height/2 + caster_height}" rpy="0 0 0" />
-      <parent link="base_footprint" />
-      <child link="base_link" />
-    </joint>
-    <xacro:wheel prefix="left" reflect="1" />
-    <xacro:wheel prefix="right" reflect="-1" />
-  </xacro:macro>
-  <!-- <xacro:shark_base/> -->
+   <!-- <link name="caster_wheel">
+     <visual>
+       <material name="darkgray"/>
+      <origin xyz="0 0 0" rpy="0 0 0"/>
+      <geometry>
+        <sphere radius="${caster_wheel_radius}"/>
+      </geometry>
+    </visual>
+    <collision>
+      <origin xyz="0 0 0" rpy="0 0 0"/>
+      <geometry>
+        <sphere radius="${caster_wheel_radius}"/>
+      </geometry>
+    </collision>
+    <xacro:sphere_inertia m="5" r="${caster_wheel_radius}"/>
+  </link>
+  <joint name="caster_wheel_joint" type="continuous">
+    <axis xyz="0 1 0" rpy="0 0 0" />
+    <parent link="base_link"/>
+    <child link="caster_wheel"/>
+    <origin xyz="${caster_wheel_joint_offset} 0 -${0.06+caster_wheel_radius}" rpy="0 0 0"/>
+  </joint> -->
 </robot>
