Commit message: :sparkles: added sick visual

File: sensors_description/urdf/sick_lms1xx.urdf.xacro (robot description, xacro)
@@ -12,7 +12,7 @@
     <link name="${name}_mount_link">
       <visual>
-        <!-- <geometry>
-          <mesh filename="/home/stihl/fbot_ws/src/sick_scan_xd/meshes/LMS1xx_small.dae" />
-        </geometry> -->
+        <geometry>
+          <mesh filename="package://sensors_description/meshes/LMS1xx_collision.stl"/>
+        </geometry>
         <material name="blue" >
           <color rgba="0 0 1 1" />
@@ -20,7 +20,7 @@
       </visual>
       <collision>
-        <!-- <geometry>
-          <mesh filename="/home/stihl/fbot_ws/src/sick_scan_xd/meshes/LMS1xx_collision.stl" />
-        </geometry> -->
+        <geometry>
+          <mesh filename="package://sensors_description/meshes/LMS1xx_small.dae"/>
+        </geometry>
       </collision>
       <inertial>

Commit message: :bug: fixed sick link position

File: sensors_description/urdf/sick_lms1xx.urdf.xacro (robot description, xacro)
@@ -13,7 +13,7 @@
       <visual>
         <geometry>
-          <mesh filename="package://sensors_description/meshes/LMS1xx_collision.stl"/>
+          <mesh filename="package://sensors_description/meshes/sick-lms1xx.stl"/>
         </geometry>
-        <material name="blue" >
+        <material name="grey" >
           <color rgba="0 0 1 1" />
         </material>
@@ -21,5 +21,5 @@
       <collision>
         <geometry>
-          <mesh filename="package://sensors_description/meshes/LMS1xx_small.dae"/>
+          <mesh filename="package://sensors_description/meshes/sick-lms1xx.dae"/>
         </geometry>
       </collision>
